Commit message: Added joint8 for gripper, and fixed controlers for joint8

File: src/piper_moveit/piper_with_gripper_moveit/config/piper.ros2_control.xacro (robot description, xacro)
@@ -57,4 +57,11 @@
                 <state_interface name="velocity"/>
             </joint>
+            <joint name="joint8">
+                <command_interface name="position"/>
+                <state_interface name="position">
+                  <param name="initial_value">${initial_positions['joint8']}</param>
+                </state_interface>
+                <state_interface name="velocity"/>
+            </joint>
         </ros2_control>
     </xacro:macro>
