Commit message: feat: improve Piper gripper sim, MoveIt config, and Gazebo URDF
Refactor joint8 gripper control, update MoveIt and ros2_control configs,
and extend Piper Gazebo world and description xacros for welding sim.

Co-authored-by: Cursor <cursoragent@cursor.com>

File: src/piper_moveit/piper_with_gripper_moveit/config/piper.ros2_control.xacro (robot description, xacro)
@@ -58,5 +58,5 @@
             </joint>
             <joint name="joint8">
-                <command_interface name="position"/>
+                <!-- URDF mimic of joint7: no command interface allowed. -->
                 <state_interface name="position">
                   <param name="initial_value">${initial_positions['joint8']}</param>

File: src/robot_description/piper_description/urdf/piper_description.xacro (robot description, xacro)
@@ -442,7 +442,9 @@
     <axis
       xyz="0 0 1" />
-    <limit
-      lower="0"
-      upper="0.035"
+    <!-- Limits match piper_description_gz.xacro so simulated joint states are
+         never out of bounds for MoveIt (sim commands open up to 0.036). -->
+    <limit
+      lower="-0.001"
+      upper="0.036"
       effort="10"
       velocity="1" />
@@ -500,12 +502,22 @@
     <axis
       xyz="0 0 -1" />
-    <limit
-      lower="-0.035"
-      upper="0"
+    <!-- Single-motor parallel jaw: joint8 physically mirrors joint7. The mimic
+         tag makes MoveIt treat the gripper group as one DOF (joint7), so RViz
+         gripper planning commands only joint7 and joint8 follows. -->
+    <mimic joint="joint7" multiplier="-1" offset="0" />
+    <limit
+      lower="-0.036"
+      upper="0.001"
       effort="10"
       velocity="1" />
   </joint>
-  <!-- MoveIt / arm_api2 TCP: tool tip offset from gripper_base (+Z), 241.1 mm. -->
-  <xacro:property name="arm_tcp_xyz" value="0 0 0.2411"/>
+  <!-- MoveIt / arm_api2 TCP: grasp point near the FINGERTIPS of the gripper
+       (gripper_base +Z; gripping region spans 0.059..0.136 m, tips ~0.136 m).
+       0.130 m sits ~6 mm inside the tips. MUST match piper_description_gz.xacro:
+       when this was 0.1 and the gz/TF model 0.130, MoveIt IK placed the real
+       fingertips 30 mm lower than planned, so the pregrasp→grasp descent drove
+       the gripper into the ground plane. (Was 0.1 finger centre, originally
+       0.2411 m — ~10 cm beyond the fingertips.) -->
+  <xacro:property name="arm_tcp_xyz" value="0 0 0.130"/>
   <link name="arm_tcp">
     <inertial>

File: src/robot_description/piper_description/urdf/piper_description_gazebo.xacro (robot description, xacro)
@@ -504,6 +504,7 @@
       velocity="1" />
   </joint>
-  <!-- MoveIt / arm_api2 TCP: tool tip offset from gripper_base (+Z), 241.1 mm. -->
-  <xacro:property name="arm_tcp_xyz" value="0 0 0.2411"/>
+  <!-- MoveIt / arm_api2 TCP: grasp point BETWEEN the two gripper fingers
+       (gripper_base +Z ~0.098 m). Was 0.2411 m, ~10 cm beyond the fingertips. -->
+  <xacro:property name="arm_tcp_xyz" value="0 0 0.1"/>
   <link name="arm_tcp">
     <inertial>

File: src/robot_description/piper_description/urdf/piper_description_gz.xacro (robot description, xacro)
@@ -446,4 +446,24 @@
           filename="file://$(find piper_description)/meshes/link7.STL" />
       </geometry>
+      <!-- High-friction, soft contact so the finger grips instead of slipping.
+           Mirrors ur_simulation_gz robotiq_2f_85_simple_parallel finger tuning. -->
+      <surface>
+        <friction>
+          <ode>
+            <mu1>100000.0</mu1>
+            <mu2>100000.0</mu2>
+          </ode>
+        </friction>
+        <contact>
+          <ode>
+            <kp>1e+5</kp>
+            <kd>1</kd>
+            <soft_cfm>0</soft_cfm>
+            <soft_erp>0.2</soft_erp>
+            <minDepth>0.002</minDepth>
+            <maxVel>0</maxVel>
+          </ode>
+        </contact>
+      </surface>
     </collision>
   </link>
@@ -461,10 +481,10 @@
       xyz="0 0 1" />
     <limit
-      lower="0"
-      upper="0.035"
+      lower="-0.001"
+      upper="0.036"
       effort="10"
       velocity="1" />
     <dynamics
-      damping="0"
+      damping="1.0"
       friction="0" />
   </joint>
@@ -507,4 +527,24 @@
           filename="file://$(find piper_description)/meshes/link8.STL" />
       </geometry>
+      <!-- High-friction, soft contact so the finger grips instead of slipping.
+           Mirrors ur_simulation_gz robotiq_2f_85_simple_parallel finger tuning. -->
+      <surface>
+        <friction>
+          <ode>
+            <mu1>100000.0</mu1>
+            <mu2>100000.0</mu2>
+          </ode>
+        </friction>
+        <contact>
+          <ode>
+            <kp>1e+5</kp>
+            <kd>1</kd>
+            <soft_cfm>0</soft_cfm>
+            <soft_erp>0.2</soft_erp>
+            <minDepth>0.002</minDepth>
+            <maxVel>0</maxVel>
+          </ode>
+        </contact>
+      </surface>
     </collision>
   </link>
@@ -521,15 +561,24 @@
     <axis
       xyz="0 0 -1" />
+    <!-- The physical gripper is a single-motor parallel jaw: joint8 always
+         mirrors joint7. gz_ros2_control (Jazzy) enforces the URDF mimic tag
+         natively, so only joint7 is commanded (no gripper8_controller and no
+         joint8_ctrl.py mirror node — that 50 Hz retriggering left joint8
+         frozen while joint7 squeezed the object alone). -->
+    <mimic joint="joint7" multiplier="-1" offset="0" />
     <limit
-      lower="-0.035"
-      upper="0"
+      lower="-0.036"
+      upper="0.001"
       effort="10"
       velocity="1" />
     <dynamics
-      damping="0"
+      damping="1.0"
       friction="0" />
   </joint>
-  <!-- MoveIt / arm_api2 TCP: tool tip offset from gripper_base (+Z), 241.1 mm. -->
-  <xacro:property name="arm_tcp_xyz" value="0 0 0.2411"/>
+  <!-- MoveIt / arm_api2 TCP: grasp point near the FINGERTIPS of the gripper
+       (gripper_base +Z; gripping region spans 0.059..0.136 m, tips ~0.136 m).
+       0.130 m sits ~6 mm inside the tips. Was 0.1 (finger centre), and
+       originally 0.2411 m (~10 cm beyond the fingertips). -->
+  <xacro:property name="arm_tcp_xyz" value="0 0 0.130"/>
   <link name="arm_tcp">
     <inertial>
@@ -580,6 +629,4 @@
       <joint name="joint1">
           <command_interface name="position"/>
-          <command_interface name="velocity"/>
-          <command_interface name="effort"/>
           <state_interface name="position">
               <param name="initial_value">0.0</param>
@@ -594,6 +641,4 @@
       <joint name="joint2">
           <command_interface name="position"/>
-          <command_interface name="velocity"/>
-          <command_interface name="effort"/>
           <state_interface name="position">
               <param name="initial_value">0.1</param>
@@ -608,6 +653,4 @@
       <joint name="joint3">
           <command_interface name="position"/>
-          <command_interface name="velocity"/>
-          <command_interface name="effort"/>
           <state_interface name="position">
               <param name="initial_value">-1.5</param>
@@ -622,6 +665,4 @@
       <joint name="joint4">
           <command_interface name="position"/>
-          <command_interface name="velocity"/>
-          <command_interface name="effort"/>
           <state_interface name="position">
               <param name="initial_value">0.0</param>
@@ -636,6 +677,4 @@
       <joint name="joint5">
           <command_interface name="position"/>
-          <command_interface name="velocity"/>
-          <command_interface name="effort"/>
           <state_interface name="position">
               <param name="initial_value">0.0</param>
@@ -650,6 +689,4 @@
       <joint name="joint6">
           <command_interface name="position"/>
-          <command_interface name="velocity"/>
-          <command_interface name="effort"/>
           <state_interface name="position">
               <param name="initial_value">0.0</param>
@@ -664,6 +701,4 @@
       <joint name="joint7">
           <command_interface name="position"/>
-          <command_interface name="velocity"/>
-          <command_interface name="effort"/>
           <state_interface name="position">
               <param name="initial_value">0.0175</param>
@@ -677,7 +712,6 @@
       </joint>
       <joint name="joint8">
-          <command_interface name="position"/>
-          <command_interface name="velocity"/>
-          <command_interface name="effort"/>
+          <!-- mimic of joint7 (see joint definition above): no command
+               interface allowed; state interfaces stay for joint_states. -->
           <state_interface name="position">
               <param name="initial_value">-0.0175</param>
