Commit message: feat: add RealSense D435 hand-eye mount macros and demo launch
Wire D435 optical frame into Piper URDF/xacro and add a demo MoveIt launch for hand-eye calibration.

Co-authored-by: Cursor <cursoragent@cursor.com>

File: src/piper_moveit/piper_with_gripper_moveit/config/piper.urdf.xacro (robot description, xacro)
@@ -2,4 +2,5 @@
 <robot xmlns:xacro="http://www.ros.org/wiki/xacro" name="piper">
     <xacro:arg name="initial_positions_file" default="initial_positions.yaml" />
+    <xacro:arg name="wrist_camera" default="oak_pro_w"/>
     <!-- Import piper urdf file -->
     <xacro:include filename="$(find piper_description)/urdf/piper_description.xacro" />

File: src/robot_description/piper_description/urdf/piper_description.xacro (robot description, xacro)
@@ -3,5 +3,8 @@
   name="piper"
   xmlns:xacro="http://ros.org/wiki/xacro">
+  <xacro:arg name="wrist_camera" default="oak_pro_w"/>
+  <xacro:property name="wrist_camera_selected" value="$(arg wrist_camera)"/>
   <xacro:include filename="$(find piper_description)/urdf/include/piper_oak_d_pro_w_handeye_macros.xacro"/>
+  <xacro:include filename="$(find piper_description)/urdf/include/piper_realsense_d435_handeye_macros.xacro"/>
 <!-- world -->
   <link name="world"/>
@@ -338,5 +341,10 @@
       velocity="3" />
   </joint>
-  <xacro:piper_mount_oak_d_pro_w_handeye parent_link="link6" simulation="false" oak_visual_mesh="true"/>
+  <xacro:if value="${wrist_camera_selected == 'realsense_d435'}">
+    <xacro:piper_mount_realsense_d435_handeye parent_link="link6" use_mesh="true"/>
+  </xacro:if>
+  <xacro:unless value="${wrist_camera_selected == 'realsense_d435'}">
+    <xacro:piper_mount_oak_d_pro_w_handeye parent_link="link6" simulation="false" oak_visual_mesh="true"/>
+  </xacro:unless>
   <link
     name="gripper_base">
