Commit message: Addedbridge camera topics from Gazebo to ROS 2 in piper_gz_sim.launch.py

File: src/robot_description/piper_description/urdf/piper_description_gazebo.xacro (robot description, xacro)
@@ -504,4 +504,69 @@
       velocity="1" />
   </joint>
+  <!-- Camera -->
+  <link name="camera_link">
+    <inertial>
+      <origin xyz="0 0 0" rpy="0 0 0" />
+      <mass value="0.01" />
+      <inertia ixx="0.00001" ixy="0.0" ixz="0.0" iyy="0.00001" iyz="0.0" izz="0.00001" />
+    </inertial>
+    <visual>
+      <origin xyz="0 0 0" rpy="0 0 0" />
+      <geometry>
+        <box size="0.02 0.04 0.02" />
+      </geometry>
+      <material name="black">
+        <color rgba="0.0 0.0 0.0 1.0" />
+      </material>
+    </visual>
+    <collision>
+      <origin xyz="0 0 0" rpy="0 0 0" />
+      <geometry>
+        <box size="0.02 0.04 0.02" />
+      </geometry>
+    </collision>
+  </link>
+  <joint name="camera_joint" type="fixed">
+    <origin xyz="0.05 0 0.02" rpy="0 0 0" />
+    <parent link="gripper_base" />
+    <child link="camera_link" />
+  </joint>
+  <!-- Gazebo camera plugin -->
+  <gazebo reference="camera_link">
+    <sensor type="camera" name="camera1">
+      <update_rate>30</update_rate>
+      <camera name="head">
+        <horizontal_fov>1.3962634</horizontal_fov>
+        <image>
+          <width>640</width>
+          <height>480</height>
+          <format>R8G8B8</format>
+        </image>
+        <clip>
+          <near>0.02</near>
+          <far>300</far>
+        </clip>
+        <noise>
+          <type>gaussian</type>
+          <mean>0.0</mean>
+          <stddev>0.007</stddev>
+        </noise>
+      </camera>
+      <plugin name="camera_controller" filename="libgazebo_ros_camera.so">
+        <alwaysOn>true</alwaysOn>
+        <updateRate>30.0</updateRate>
+        <cameraName>piper/camera</cameraName>
+        <imageTopicName>image_raw</imageTopicName>
+        <cameraInfoTopicName>camera_info</cameraInfoTopicName>
+        <frameName>camera_link</frameName>
+        <hackBaseline>0.07</hackBaseline>
+        <distortionK1>0.0</distortionK1>
+        <distortionK2>0.0</distortionK2>
+        <distortionK3>0.0</distortionK3>
+        <distortionT1>0.0</distortionT1>
+        <distortionT2>0.0</distortionT2>
+      </plugin>
+    </sensor>
+  </gazebo>
   <!-- <gazebo reference="base_link">
       <material>Gazebo/Black</material>

File: src/robot_description/piper_description/urdf/piper_description_gz.xacro (robot description, xacro)
@@ -675,3 +675,56 @@
       </joint>
   </ros2_control>
+  <!-- Camera -->
+  <link name="camera_link">
+    <inertial>
+      <origin xyz="0 0 0" rpy="0 0 0" />
+      <mass value="0.01" />
+      <inertia ixx="0.00001" ixy="0.0" ixz="0.0" iyy="0.00001" iyz="0.0" izz="0.00001" />
+    </inertial>
+    <visual>
+      <origin xyz="0 0 0" rpy="0 0 0" />
+      <geometry>
+        <box size="0.02 0.04 0.02" />
+      </geometry>
+      <material>
+        <color rgba="0.0 0.0 0.0 1.0" />
+      </material>
+    </visual>
+    <collision>
+      <origin xyz="0 0 0" rpy="0 0 0" />
+      <geometry>
+        <box size="0.02 0.04 0.02" />
+      </geometry>
+    </collision>
+  </link>
+  <joint name="camera_joint" type="revolute">
+    <parent link="gripper_base"/>
+    <child link="camera_link"/>
+    <origin xyz="-0.05 0 0.02" rpy="0 -1.5708 0"/>
+    <!-- Rotation around Z axis -->
+    <axis xyz="0 0 1"/>
+    <!-- Realistic limits (≈ ±90°) -->
+    <limit lower="-1.57" upper="1.57" effort="10.0" velocity="1.0"/>
+    <!-- Prevent numerical jitter -->
+    <dynamics damping="0.1" friction="0.0"/>
+  </joint>
+  <!-- Gazebo (Gz) camera sensor -->
+  <gazebo reference="camera_link">
+    <sensor name="camera" type="camera">
+      <camera>
+        <horizontal_fov>1.3962634</horizontal_fov>
+        <image>
+          <width>640</width>
+          <height>480</height>
+        </image>
+        <clip>
+          <near>0.02</near>
+          <far>300</far>
+        </clip>
+      </camera>
+      <always_on>1</always_on>
+      <update_rate>30</update_rate>
+      <visualize>true</visualize>
+    </sensor>
+  </gazebo>
 </robot>
