Commit message: Piper fixed in gazebo

File: src/robot_description/piper_description/urdf/piper_description_gz.xacro (robot description, xacro)
@@ -15,5 +15,5 @@
             <origin xyz="-0.00473641164191482 2.56829134630247E-05 0.041451518036016" rpy="0 0 0" />
             <mass value="1.02" />
-            <inertia ixx="0.00267433" ixy="-0.00000073" ixz="-0.00017389" iyy="0.00282612" iyz="0.0000004" izz="0.00089624" />
+            <inertia ixx="0.0001" ixy="0.0" ixz="0.0" iyy="0.0001" iyz="0.0" izz="0.0001" />
     </inertial>
     <visual>
@@ -46,5 +46,5 @@
             <origin xyz="0.000121504734057468 0.000104632162460536 -0.00438597309559853" rpy="0 0 0" />
             <mass value="0.71" />
-            <inertia ixx="0.00048916" ixy="-0.00000036" ixz="-0.00000224" iyy="0.00040472" iyz="-0.00000242" izz="0.00043982" />
+            <inertia ixx="0.0001" ixy="0.0" ixz="0.0" iyy="0.0001" iyz="0.0" izz="0.0001" />
     </inertial>
     <visual>
@@ -89,4 +89,7 @@
       effort="100"
       velocity="5" />
+    <dynamics
+      damping="0"
+      friction="0" />
   </joint>
   <link
@@ -95,5 +98,5 @@
             <origin xyz="0.198666145229743 -0.010926924140076 0.00142121714502687" rpy="0 0 0" />
             <mass value="1.17" />
-            <inertia ixx="0.00116918" ixy="-0.00180037" ixz="0.00025146" iyy="0.06785384" iyz="-0.00000455" izz="0.06774489" />
+            <inertia ixx="0.0001" ixy="0.0" ixz="0.0" iyy="0.0001" iyz="0.0" izz="0.0001" />
     </inertial>
     <visual>
@@ -139,4 +142,7 @@
       effort="100"
       velocity="5" />
+    <dynamics
+      damping="0"
+      friction="0" />
   </joint>
   <link
@@ -145,5 +151,5 @@
             <origin xyz="-0.0202737662122021 -0.133914995944595 -0.000458682652737356" rpy="0 0 0" />
             <mass value="0.5" />
-            <inertia ixx="0.01361711" ixy="0.00165794" ixz="-0.00000048" iyy="0.00045024" iyz="-0.00000045" izz="0.01380322" />
+            <inertia ixx="0.0001" ixy="0.0" ixz="0.0" iyy="0.0001" iyz="0.0" izz="0.0001" />
     </inertial>
     <visual>
@@ -189,4 +195,7 @@
       effort="100"
       velocity="5" />
+    <dynamics
+      damping="0"
+      friction="0" />
   </joint>
   <link
@@ -195,5 +204,5 @@
             <origin xyz="-9.66635791618542E-05 0.000876064475651083 -0.00496880904640868" rpy="0 0 0" />
             <mass value="0.38" />
-            <inertia ixx="0.00018501" ixy="0.00000054" ixz="0.00000120" iyy="0.00018965" iyz="-0.00000841" izz="0.00015484" />
+            <inertia ixx="0.0001" ixy="0.0" ixz="0.0" iyy="0.0001" iyz="0.0" izz="0.0001" />
     </inertial>
     <visual>
@@ -238,4 +247,7 @@
       effort="100"
       velocity="5" />
+    <dynamics
+      damping="0"
+      friction="0" />
   </joint>
   <link
@@ -244,5 +256,5 @@
             <origin xyz="-4.10554118924211E-05 -0.0566486692356075 -0.0037205791677906" rpy="0 0 0" />
             <mass value="0.383" />
-            <inertia ixx="0.00166169" ixy="0.00000006" ixz="-0.00000007" iyy="0.00018510" iyz="0.00001026" izz="0.00164321" />
+            <inertia ixx="0.0001" ixy="0.0" ixz="0.0" iyy="0.0001" iyz="0.0" izz="0.0001" />
     </inertial>
     <visual>
@@ -287,4 +299,7 @@
       effort="100"
       velocity="5" />
+    <dynamics
+      damping="0"
+      friction="0" />
   </joint>
   <link
@@ -293,5 +308,5 @@
             <origin xyz="-8.82590762930069E-05 9.0598378529832E-06 -0.002" rpy="0 0 0" />
             <mass value="0.00699089613564366" />
-            <inertia ixx="5.73015540542155E-07" ixy="-1.98305403089247E-22" ixz="-7.2791893904596E-23" iyy="5.73015540542155E-07" iyz="-3.4146026640245E-24" izz="1.06738869138926E-06" />
+            <inertia ixx="0.00001" ixy="0.0" ixz="0.0" iyy="0.00001" iyz="0.0" izz="0.00001" />
     </inertial>
     <visual>
@@ -336,4 +351,7 @@
       effort="100"
       velocity="3" />
+    <dynamics
+      damping="0"
+      friction="0" />
   </joint>
   <link
@@ -346,10 +364,10 @@
         value="0.45" />
       <inertia
-        ixx="0.00092934"
-        ixy="0.00000034"
-        ixz="-0.00000738"
-        iyy="0.00071447"
-        iyz="0.00000005"
-        izz="0.00039442" />
+        ixx="0.0001"
+        ixy="0.0"
+        ixz="0.0"
+        iyy="0.0001"
+        iyz="0.0"
+        izz="0.0001" />
     </inertial>
     <visual>
@@ -397,10 +415,10 @@
         value="0.025" />
       <inertia
-        ixx="0.00007371"
-        ixy="-0.00000113"
-        ixz="0.00000021"
-        iyy="0.00007371"
-        iyz="-0.00001372"
-        izz="0.0000747" />
+        ixx="0.00001"
+        ixy="0.0"
+        ixz="0.0"
+        iyy="0.00001"
+        iyz="0.0"
+        izz="0.00001" />
     </inertial>
     <visual>
@@ -445,4 +463,7 @@
       effort="10"
       velocity="1" />
+    <dynamics
+      damping="0"
+      friction="0" />
   </joint>
   <link
@@ -455,10 +476,10 @@
         value="0.025" />
       <inertia
-        ixx="0.00007371"
-        ixy="-0.00000113"
-        ixz="0.00000021"
-        iyy="0.00007371"
-        iyz="-0.00001372"
-        izz="0.0000747" />
+        ixx="0.00001"
+        ixy="0.0"
+        ixz="0.0"
+        iyy="0.00001"
+        iyz="0.0"
+        izz="0.00001" />
     </inertial>
     <visual>
@@ -503,36 +524,38 @@
       effort="10"
       velocity="1" />
-  </joint>
-  <!-- <gazebo reference="base_link">
-      <material>Gazebo/Black</material>
-      <gravity>true</gravity>
+    <dynamics
+      damping="0"
+      friction="0" />
+  </joint>
+  <gazebo reference="base_link">
       <selfCollide>false</selfCollide>
   </gazebo>
   <gazebo reference="link1">
-      <material>Gazebo/Gray</material>
       <selfCollide>false</selfCollide>
   </gazebo>
   <gazebo reference="link2">
-      <material>Gazebo/Red</material>
       <selfCollide>false</selfCollide>
   </gazebo>
   <gazebo reference="link3">
-      <material>Gazebo/Blue</material>
+      <selfCollide>false</selfCollide>
   </gazebo>
   <gazebo reference="link4">
-      <material>Gazebo/Green</material>
+      <selfCollide>false</selfCollide>
   </gazebo>
   <gazebo reference="link5">
-      <material>Gazebo/Yellow</material>
+      <selfCollide>false</selfCollide>
   </gazebo>
   <gazebo reference="link6">
-      <material>Gazebo/Orange</material>
+      <selfCollide>false</selfCollide>
+  </gazebo>
+  <gazebo reference="gripper_base">
+      <selfCollide>false</selfCollide>
   </gazebo>
   <gazebo reference="link7">
-      <material>Gazebo/Orange</material>
+      <selfCollide>false</selfCollide>
   </gazebo>
   <gazebo reference="link8">
-      <material>Gazebo/Orange</material>
-  </gazebo> -->
+      <selfCollide>false</selfCollide>
+  </gazebo>
   <ros2_control name="GazeboSimSystem" type="system">
       <hardware>
@@ -540,82 +563,114 @@
       </hardware>
       <joint name="joint1">
-          <command_interface name="position">
-              <param name="min">-1</param>
-              <param name="max">1</param>
-          </command_interface>
-          <state_interface name="position">
-              <param name="initial_value">0.0</param>
-          </state_interface>
-          <state_interface name="velocity"/>
+          <command_interface name="position"/>
+          <command_interface name="velocity"/>
+          <command_interface name="effort"/>
+          <state_interface name="position">
+              <param name="initial_value">0.0</param>
+          </state_interface>
+          <state_interface name="velocity">
+              <param name="initial_value">0.0</param>
+          </state_interface>
+          <state_interface name="effort">
+              <param name="initial_value">0.0</param>
+          </state_interface>
       </joint>
       <joint name="joint2">
-          <command_interface name="position">
-              <param name="min">-1</param>
-              <param name="max">1</param>
-          </command_interface>
-          <state_interface name="position">
-              <param name="initial_value">0.0</param>
-          </state_interface>
-          <state_interface name="velocity"/>
+          <command_interface name="position"/>
+          <command_interface name="velocity"/>
+          <command_interface name="effort"/>
+          <state_interface name="position">
+              <param name="initial_value">0.1</param>
+          </state_interface>
+          <state_interface name="velocity">
+              <param name="initial_value">0.0</param>
+          </state_interface>
+          <state_interface name="effort">
+              <param name="initial_value">0.0</param>
+          </state_interface>
       </joint>
       <joint name="joint3">
-          <command_interface name="position">
-              <param name="min">-1</param>
-              <param name="max">1</param>
-          </command_interface>
-          <state_interface name="position">
-              <param name="initial_value">0.0</param>
-          </state_interface>
-          <state_interface name="velocity"/>
+          <command_interface name="position"/>
+          <command_interface name="velocity"/>
+          <command_interface name="effort"/>
+          <state_interface name="position">
+              <param name="initial_value">-1.5</param>
+          </state_interface>
+          <state_interface name="velocity">
+              <param name="initial_value">0.0</param>
+          </state_interface>
+          <state_interface name="effort">
+              <param name="initial_value">0.0</param>
+          </state_interface>
       </joint>
       <joint name="joint4">
-          <command_interface name="position">
-              <param name="min">-1</param>
-              <param name="max">1</param>
-          </command_interface>
-          <state_interface name="position">
-              <param name="initial_value">0.0</param>
-          </state_interface>
-          <state_interface name="velocity"/>
+          <command_interface name="position"/>
+          <command_interface name="velocity"/>
+          <command_interface name="effort"/>
+          <state_interface name="position">
+              <param name="initial_value">0.0</param>
+          </state_interface>
+          <state_interface name="velocity">
+              <param name="initial_value">0.0</param>
+          </state_interface>
+          <state_interface name="effort">
+              <param name="initial_value">0.0</param>
+          </state_interface>
       </joint>
       <joint name="joint5">
-          <command_interface name="position">
-              <param name="min">-1</param>
-              <param name="max">1</param>
-          </command_interface>
-          <state_interface name="position">
-              <param name="initial_value">0.0</param>
-          </state_interface>
-          <state_interface name="velocity"/>
+          <command_interface name="position"/>
+          <command_interface name="velocity"/>
+          <command_interface name="effort"/>
+          <state_interface name="position">
+              <param name="initial_value">0.0</param>
+          </state_interface>
+          <state_interface name="velocity">
+              <param name="initial_value">0.0</param>
+          </state_interface>
+          <state_interface name="effort">
+              <param name="initial_value">0.0</param>
+          </state_interface>
       </joint>
       <joint name="joint6">
-          <command_interface name="position">
-              <param name="min">-1</param>
-              <param name="max">1</param>
-          </command_interface>
-          <state_interface name="position">
-              <param name="initial_value">0.0</param>
-          </state_interface>
-          <state_interface name="velocity"/>
+          <command_interface name="position"/>
+          <command_interface name="velocity"/>
+          <command_interface name="effort"/>
+          <state_interface name="position">
+              <param name="initial_value">0.0</param>
+          </state_interface>
+          <state_interface name="velocity">
+              <param name="initial_value">0.0</param>
+          </state_interface>
+          <state_interface name="effort">
+              <param name="initial_value">0.0</param>
+          </state_interface>
       </joint>
       <joint name="joint7">
-          <command_interface name="position">
-              <param name="min">-1</param>
-              <param name="max">1</param>
-          </command_interface>
-          <state_interface name="position">
-              <param name="initial_value">0.0</param>
-          </state_interface>
-          <state_interface name="velocity"/>
+          <command_interface name="position"/>
+          <command_interface name="velocity"/>
+          <command_interface name="effort"/>
+          <state_interface name="position">
+              <param name="initial_value">0.0175</param>
+          </state_interface>
+          <state_interface name="velocity">
+              <param name="initial_value">0.0</param>
+          </state_interface>
+          <state_interface name="effort">
+              <param name="initial_value">0.0</param>
+          </state_interface>
       </joint>
       <joint name="joint8">
-          <command_interface name="position">
-              <param name="min">-1</param>
-              <param name="max">1</param>
-          </command_interface>
-          <state_interface name="position">
-              <param name="initial_value">0.0</param>
-          </state_interface>
-          <state_interface name="velocity"/>
+          <command_interface name="position"/>
+          <command_interface name="velocity"/>
+          <command_interface name="effort"/>
+          <state_interface name="position">
+              <param name="initial_value">-0.0175</param>
+          </state_interface>
+          <state_interface name="velocity">
+              <param name="initial_value">0.0</param>
+          </state_interface>
+          <state_interface name="effort">
+              <param name="initial_value">0.0</param>
+          </state_interface>
       </joint>
   </ros2_control>

Commit message: feat: add RGB-D camera support with depth/point cloud bridging and MoveIt fixes
Camera & Sensor Changes:
- Upgrade camera to RGB-D sensor in Gazebo Sim with depth output
- Add ros_gz_image bridge for depth image with 32FC1 format
- Add depth_to_uint16.py converter for RViz-compatible 16UC1 depth images
- Add pointcloud_reframe.py to republish point cloud with correct frame_id
- Change camera_joint to fixed joint for consistent TF publishing
- Add static TF publishers for camera frame transforms

MoveIt Configuration:
- Remove gripper kinematics config (not a kinematic chain)

RViz Stability:
- Add QT_QPA_PLATFORM=xcb and software rendering for RViz GL compatibility

Launch & Build:
- Update piper_gz_sim.launch.py with Beer can spawning and GZ_SIM_RESOURCE_PATH
- Add rclpy and numpy dependencies to piper_gazebo package
- Install new depth and point cloud processing scripts

File: src/robot_description/piper_description/urdf/piper_description_gz.xacro (robot description, xacro)
@@ -687,5 +687,5 @@
         <box size="0.02 0.04 0.02" />
       </geometry>
-      <material>
+      <material name="camera_black">
         <color rgba="0.0 0.0 0.0 1.0" />
       </material>
@@ -698,18 +698,12 @@
     </collision>
   </link>
-  <joint name="camera_joint" type="revolute">
+  <joint name="camera_joint" type="fixed">
     <parent link="gripper_base"/>
     <child link="camera_link"/>
     <origin xyz="-0.05 0 0.02" rpy="0 -1.5708 0"/>
-    <!-- Rotation around Z axis -->
-    <axis xyz="0 0 1"/>
-    <!-- Realistic limits (≈ ±90°) -->
-    <limit lower="-1.57" upper="1.57" effort="10.0" velocity="1.0"/>
-    <!-- Prevent numerical jitter -->
-    <dynamics damping="0.1" friction="0.0"/>
-  </joint>
-  <!-- Gazebo (Gz) camera sensor -->
+  </joint>
+  <!-- Gazebo (Gz) RGB-D camera sensor -->
   <gazebo reference="camera_link">
-    <sensor name="camera" type="camera">
+    <sensor name="camera" type="rgbd_camera">
       <camera>
         <horizontal_fov>1.3962634</horizontal_fov>
@@ -723,4 +717,16 @@
         </clip>
       </camera>
+      <depth_camera>
+        <image>
+          <width>640</width>
+          <height>480</height>
+          <format>R_FLOAT32</format>
+        </image>
+        <clip>
+          <near>0.02</near>
+          <far>10.0</far>
+        </clip>
+        <point_cloud>true</point_cloud>
+      </depth_camera>
       <always_on>1</always_on>
       <update_rate>30</update_rate>

Commit message: Added RGBD camera, banana and can model to the sceeen, and an aeuco marker. Aruco poze estimation and Hand-eye-calibration still fail

File: src/robot_description/piper_description/urdf/piper_description_gz.xacro (robot description, xacro)
@@ -699,5 +699,5 @@
   </link>
   <joint name="camera_joint" type="fixed">
-    <parent link="gripper_base"/>
+    <parent link="link6"/>
     <child link="camera_link"/>
     <origin xyz="-0.05 0 0.02" rpy="0 -1.5708 0"/>
@@ -734,3 +734,18 @@
     </sensor>
   </gazebo>
+  <!-- Camera optical frame (ROS convention: X right, Y down, Z forward) -->
+  <link name="camera_optical_frame">
+    <inertial>
+      <origin xyz="0 0 0" rpy="0 0 0" />
+      <mass value="0.0001" />
+      <inertia ixx="0.00000001" ixy="0.0" ixz="0.0" iyy="0.00000001" iyz="0.0" izz="0.00000001" />
+    </inertial>
+  </link>
+  <joint name="camera_optical_joint" type="fixed">
+    <parent link="camera_link"/>
+    <child link="camera_optical_frame"/>
+    <!-- optical: X right, Y down, Z forward (ROS REP 103 standard) -->
+    <!-- This is independent of camera mount - converts to optical convention -->
+    <origin xyz="0 0 0" rpy="-1.57079632679 0 -1.57079632679"/>
+  </joint>
 </robot>

Commit message: added models, floor and aruco marker

File: src/robot_description/piper_description/urdf/piper_description_gz.xacro (robot description, xacro)
@@ -701,5 +701,5 @@
     <parent link="link6"/>
     <child link="camera_link"/>
-    <origin xyz="-0.05 0 0.02" rpy="0 -1.5708 0"/>
+    <origin xyz="-0.05 0 0" rpy="0 -1.5708 0"/>
   </joint>
   <!-- Gazebo (Gz) RGB-D camera sensor -->
@@ -745,7 +745,8 @@
     <parent link="camera_link"/>
     <child link="camera_optical_frame"/>
-    <!-- optical: X right, Y down, Z forward (ROS REP 103 standard) -->
-    <!-- This is independent of camera mount - converts to optical convention -->
-    <origin xyz="0 0 0" rpy="-1.57079632679 0 -1.57079632679"/>
+    <!--
+      ros and gazebo convenntions don align
+    -->
+    <origin xyz="0 0 0" rpy="-1.5708 0 -1.5708"/>
   </joint>
 </robot>
