Commit message: feat(gazebo,urdf): RGB-D hand-eye xacro, no-gripper Gazebo model, sim launch updates
Merge line includes prior integration with apirsic/devel2 MoveIt joint limits;
this commit adds Oak hand-eye macros, no-gripper gz description and launch,
bridge and SRDF tweaks, and documentation updates.

Co-authored-by: Cursor <cursoragent@cursor.com>

File: src/robot_description/piper_description/urdf/piper_description.xacro (robot description, xacro)
@@ -3,4 +3,5 @@
   name="piper"
   xmlns:xacro="http://ros.org/wiki/xacro">
+  <xacro:include filename="$(find piper_description)/urdf/include/piper_oak_d_sr_handeye_macros.xacro"/>
 <!-- world -->
   <link name="world"/>
@@ -337,4 +338,5 @@
       velocity="3" />
   </joint>
+  <xacro:piper_mount_oak_d_sr_handeye parent_link="link6" simulation="false" oak_gazebo_rgbd_sensor="false"/>
   <link
     name="gripper_base">

File: src/robot_description/piper_description/urdf/piper_no_gripper_description.xacro (robot description, xacro)
@@ -3,4 +3,5 @@
   name="piper"
   xmlns:xacro="http://ros.org/wiki/xacro">
+  <xacro:include filename="$(find piper_description)/urdf/include/piper_oak_d_sr_handeye_macros.xacro"/>
 <!-- world -->
   <link name="world"/>
@@ -337,4 +338,5 @@
       velocity="5" />
   </joint>
+  <xacro:piper_mount_oak_d_sr_handeye parent_link="link6" simulation="false" oak_gazebo_rgbd_sensor="false"/>
 <!-- controller -->
   <xacro:macro name="transmission_block" params="tran_name joint_name motor_name">

File: src/robot_description/piper_description/urdf/piper_no_gripper_description_gz.xacro (robot description, xacro)
@@ -15,5 +15,5 @@
             <origin xyz="-0.00473641164191482 2.56829134630247E-05 0.041451518036016" rpy="0 0 0" />
             <mass value="1.02" />
-            <inertia ixx="0.0001" ixy="0.0" ixz="0.0" iyy="0.0001" iyz="0.0" izz="0.0001" />
+            <inertia ixx="0.00267433" ixy="-0.00000073" ixz="-0.00017389" iyy="0.00282612" iyz="0.0000004" izz="0.00089624" />
     </inertial>
     <visual>
@@ -46,5 +46,5 @@
             <origin xyz="0.000121504734057468 0.000104632162460536 -0.00438597309559853" rpy="0 0 0" />
             <mass value="0.71" />
-            <inertia ixx="0.0001" ixy="0.0" ixz="0.0" iyy="0.0001" iyz="0.0" izz="0.0001" />
+            <inertia ixx="0.00048916" ixy="-0.00000036" ixz="-0.00000224" iyy="0.00040472" iyz="-0.00000242" izz="0.00043982" />
     </inertial>
     <visual>
@@ -89,7 +89,4 @@
       effort="100"
       velocity="5" />
-    <dynamics
-      damping="0"
-      friction="0" />
   </joint>
   <link
@@ -98,5 +95,5 @@
             <origin xyz="0.198666145229743 -0.010926924140076 0.00142121714502687" rpy="0 0 0" />
             <mass value="1.17" />
-            <inertia ixx="0.0001" ixy="0.0" ixz="0.0" iyy="0.0001" iyz="0.0" izz="0.0001" />
+            <inertia ixx="0.00116918" ixy="-0.00180037" ixz="0.00025146" iyy="0.06785384" iyz="-0.00000455" izz="0.06774489" />
     </inertial>
     <visual>
@@ -130,5 +127,4 @@
       xyz="0 0 0"
       rpy="1.5708 -0.1359 -3.1416" />
-      <!-- rpy="1.5708 -0.10095-0.03490659 -3.1416" /> -->
     <parent
       link="link1" />
@@ -142,7 +138,4 @@
       effort="100"
       velocity="5" />
-    <dynamics
-      damping="0"
-      friction="0" />
   </joint>
   <link
@@ -151,5 +144,5 @@
             <origin xyz="-0.0202737662122021 -0.133914995944595 -0.000458682652737356" rpy="0 0 0" />
             <mass value="0.5" />
-            <inertia ixx="0.0001" ixy="0.0" ixz="0.0" iyy="0.0001" iyz="0.0" izz="0.0001" />
+            <inertia ixx="0.01361711" ixy="0.00165794" ixz="-0.00000048" iyy="0.00045024" iyz="-0.00000045" izz="0.01380322" />
     </inertial>
     <visual>
@@ -183,5 +176,4 @@
       xyz="0.28503 0 0"
       rpy="0 0 -1.7939" />
-      <!-- rpy="0 0 -1.759-0.03490659" /> -->
     <parent
       link="link2" />
@@ -195,7 +187,4 @@
       effort="100"
       velocity="5" />
-    <dynamics
-      damping="0"
-      friction="0" />
   </joint>
   <link
@@ -204,5 +193,5 @@
             <origin xyz="-9.66635791618542E-05 0.000876064475651083 -0.00496880904640868" rpy="0 0 0" />
             <mass value="0.38" />
-            <inertia ixx="0.0001" ixy="0.0" ixz="0.0" iyy="0.0001" iyz="0.0" izz="0.0001" />
+            <inertia ixx="0.00018501" ixy="0.00000054" ixz="0.00000120" iyy="0.00018965" iyz="-0.00000841" izz="0.00015484" />
     </inertial>
     <visual>
@@ -247,7 +236,4 @@
       effort="100"
       velocity="5" />
-    <dynamics
-      damping="0"
-      friction="0" />
   </joint>
   <link
@@ -256,5 +242,5 @@
             <origin xyz="-4.10554118924211E-05 -0.0566486692356075 -0.0037205791677906" rpy="0 0 0" />
             <mass value="0.383" />
-            <inertia ixx="0.0001" ixy="0.0" ixz="0.0" iyy="0.0001" iyz="0.0" izz="0.0001" />
+            <inertia ixx="0.00166169" ixy="0.00000006" ixz="-0.00000007" iyy="0.00018510" iyz="0.00001026" izz="0.00164321" />
     </inertial>
     <visual>
@@ -299,7 +285,4 @@
       effort="100"
       velocity="5" />
-    <dynamics
-      damping="0"
-      friction="0" />
   </joint>
   <link
@@ -308,5 +291,5 @@
             <origin xyz="-8.82590762930069E-05 9.0598378529832E-06 -0.002" rpy="0 0 0" />
             <mass value="0.00699089613564366" />
-            <inertia ixx="0.00001" ixy="0.0" ixz="0.0" iyy="0.00001" iyz="0.0" izz="0.00001" />
+            <inertia ixx="5.73015540542155E-07" ixy="-1.98305403089247E-22" ixz="-7.2791893904596E-23" iyy="5.73015540542155E-07" iyz="-3.4146026640245E-24" izz="1.06738869138926E-06" />
     </inertial>
     <visual>
@@ -351,183 +334,7 @@
       effort="100"
       velocity="3" />
-    <dynamics
-      damping="0"
-      friction="0" />
   </joint>
   <xacro:include filename="$(find piper_description)/urdf/include/piper_oak_d_sr_handeye_macros.xacro"/>
   <xacro:piper_mount_oak_d_sr_handeye parent_link="link6" simulation="true" oak_gazebo_rgbd_sensor="true"/>
-  <link
-    name="gripper_base">
-    <inertial>
-      <origin
-        xyz="-0.000183807162235591 8.05033155577911E-05 0.0321436689908876"
-        rpy="0 0 0" />
-      <mass
-        value="0.45" />
-      <inertia
-        ixx="0.0001"
-        ixy="0.0"
-        ixz="0.0"
-        iyy="0.0001"
-        iyz="0.0"
-        izz="0.0001" />
-    </inertial>
-    <visual>
-      <origin
-        xyz="0 0 0"
-        rpy="0 0 0" />
-      <geometry>
-        <mesh
-          filename="file://$(find piper_description)/meshes/gripper_base.STL" />
-      </geometry>
-      <material
-        name="">
-        <color
-          rgba="0.792156862745098 0.819607843137255 0.933333333333333 1" />
-      </material>
-    </visual>
-    <collision>
-      <origin
-        xyz="0 0 0"
-        rpy="0 0 0" />
-      <geometry>
-        <mesh
-          filename="file://$(find piper_description)/meshes/gripper_base.STL" />
-      </geometry>
-    </collision>
-  </link>
-  <joint
-    name="joint6_to_gripper_base"
-    type="fixed">
-    <origin
-      xyz="0 0 0"
-      rpy="0 0 0" />
-    <parent
-      link="link6" />
-    <child
-      link="gripper_base" />
-  </joint>
-  <link
-    name="link7">
-    <inertial>
-      <origin
-        xyz="0.00065123185041968 -0.0491929869131989 0.00972258769184025"
-        rpy="0 0 0" />
-      <mass
-        value="0.025" />
-      <inertia
-        ixx="0.00001"
-        ixy="0.0"
-        ixz="0.0"
-        iyy="0.00001"
-        iyz="0.0"
-        izz="0.00001" />
-    </inertial>
-    <visual>
-      <origin
-        xyz="0 0 0"
-        rpy="0 0 0" />
-      <geometry>
-        <mesh
-          filename="file://$(find piper_description)/meshes/link7.STL" />
-      </geometry>
-      <material
-        name="">
-        <color
-          rgba="0.792156862745098 0.819607843137255 0.933333333333333 1" />
-      </material>
-    </visual>
-    <collision>
-      <origin
-        xyz="0 0 0"
-        rpy="0 0 0" />
-      <geometry>
-        <mesh
-          filename="file://$(find piper_description)/meshes/link7.STL" />
-      </geometry>
-    </collision>
-  </link>
-  <joint
-    name="joint7"
-    type="prismatic">
-    <origin
-      xyz="0 0 0.1358"
-      rpy="1.5708 0 0" />
-    <parent
-      link="gripper_base" />
-    <child
-      link="link7" />
-    <axis
-      xyz="0 0 1" />
-    <limit
-      lower="0"
-      upper="0.035"
-      effort="10"
-      velocity="1" />
-    <dynamics
-      damping="0"
-      friction="0" />
-  </joint>
-  <link
-    name="link8">
-    <inertial>
-      <origin
-        xyz="0.000651231850419722 -0.0491929869131991 0.00972258769184024"
-        rpy="0 0 0" />
-      <mass
-        value="0.025" />
-      <inertia
-        ixx="0.00001"
-        ixy="0.0"
-        ixz="0.0"
-        iyy="0.00001"
-        iyz="0.0"
-        izz="0.00001" />
-    </inertial>
-    <visual>
-      <origin
-        xyz="0 0 0"
-        rpy="0 0 0" />
-      <geometry>
-        <mesh
-          filename="file://$(find piper_description)/meshes/link8.STL" />
-      </geometry>
-      <material
-        name="">
-        <color
-          rgba="0.792156862745098 0.819607843137255 0.933333333333333 1" />
-      </material>
-    </visual>
-    <collision>
-      <origin
-        xyz="0 0 0"
-        rpy="0 0 0" />
-      <geometry>
-        <mesh
-          filename="file://$(find piper_description)/meshes/link8.STL" />
-      </geometry>
-    </collision>
-  </link>
-  <joint
-    name="joint8"
-    type="prismatic">
-    <origin
-      xyz="0 0 0.1358"
-      rpy="1.5708 0 -3.1416" />
-    <parent
-      link="gripper_base" />
-    <child
-      link="link8" />
-    <axis
-      xyz="0 0 -1" />
-    <limit
-      lower="-0.035"
-      upper="0"
-      effort="10"
-      velocity="1" />
-    <dynamics
-      damping="0"
-      friction="0" />
-  </joint>
   <gazebo reference="base_link">
       <selfCollide>false</selfCollide>
@@ -549,13 +356,4 @@
   </gazebo>
   <gazebo reference="link6">
-      <selfCollide>false</selfCollide>
-  </gazebo>
-  <gazebo reference="gripper_base">
-      <selfCollide>false</selfCollide>
-  </gazebo>
-  <gazebo reference="link7">
-      <selfCollide>false</selfCollide>
-  </gazebo>
-  <gazebo reference="link8">
       <selfCollide>false</selfCollide>
   </gazebo>
@@ -648,32 +446,4 @@
           </state_interface>
       </joint>
-      <joint name="joint7">
-          <command_interface name="position"/>
-          <command_interface name="velocity"/>
-          <command_interface name="effort"/>
-          <state_interface name="position">
-              <param name="initial_value">0.0175</param>
-          </state_interface>
-          <state_interface name="velocity">
-              <param name="initial_value">0.0</param>
-          </state_interface>
-          <state_interface name="effort">
-              <param name="initial_value">0.0</param>
-          </state_interface>
-      </joint>
-      <joint name="joint8">
-          <command_interface name="position"/>
-          <command_interface name="velocity"/>
-          <command_interface name="effort"/>
-          <state_interface name="position">
-              <param name="initial_value">-0.0175</param>
-          </state_interface>
-          <state_interface name="velocity">
-              <param name="initial_value">0.0</param>
-          </state_interface>
-          <state_interface name="effort">
-              <param name="initial_value">0.0</param>
-          </state_interface>
-      </joint>
   </ros2_control>
 </robot>
