Commit message: .

File: src/robot_description/piper_description/urdf/piper_description.xacro (robot description, xacro)
@@ -400,5 +400,5 @@
         ixy="-0.00000113"
         ixz="0.00000021"
-        iyy="-0.00000113"
+        iyy="0.00007371"
         iyz="-0.00001372"
         izz="0.0000747" />
@@ -458,5 +458,5 @@
         ixy="-0.00000113"
         ixz="0.00000021"
-        iyy="-0.00000113"
+        iyy="0.00007371"
         iyz="-0.00001372"
         izz="0.0000747" />

File: src/robot_description/piper_description/urdf/piper_description_gz.xacro (robot description, xacro)
@@ -701,5 +701,5 @@
     <parent link="link6"/>
     <child link="camera_link"/>
-    <origin xyz="-0.05 0 0" rpy="0 -1.5708 0"/>
+    <origin xyz="-0.1 0 0" rpy="0 -1.5708 0"/>
   </joint>
   <!-- Gazebo (Gz) RGB-D camera sensor -->
