Commit message: piper description for simulation

File: src/robot_description/piper_description/urdf/include/piper_oak_d_sr_handeye_macros.xacro (robot description, xacro)
@@ -8,21 +8,29 @@
   where T_nominal = trans(0,-0.01,0) × rot(rpy = -π/2, 0, -π/2 intrinsic xyz, same convention as depthai_macro).
   If you save a NEW calibration or change camera_model, recreate the fixed joint numeric values this way.
-  Values below match ~/.ros/hand_eye_calibration.yaml on this workspace (tracking_base=oak_right_camera_optical_frame).
+  Updated from saved YAML (handeye_depthai_mount_args / same T_mount math).
+  piper_description.xacro passes oak_visual_mesh:=false for MoveIt/RViz (no depthai STL mesh; TF unchanged).
   Still do not run hand_eye_calibration/publish.launch simultaneously (duplicate TF).
-  Corrected link6 → oak-d-base-frame (REP-103 URDF roll-pitch-yaw = intrinsic XYZ, same as depthai_joint rpy fields):
-    xyz = -0.068133439 0.007721162 0.055194547
-    rpy = +0.17430916 -1.23276438 -0.22762161
+  Hand-eye estimate (link6→oak_right_camera_optical_frame): tx ty tz qx qy qz qw =
+    -0.0916 -0.0015 0.0632 0.1157 -0.1322 0.7206 -0.6708
+  link6 → oak-d-base-frame (REP-103 URDF roll-pitch-yaw = intrinsic XYZ):
+    xyz = -0.090866253 0.008472480 0.063306116
+    rpy = 0.030685051 -1.217622058 -0.102237087
 -->
 <robot xmlns:xacro="http://ros.org/wiki/xacro" name="piper_oak_attachment_defs">
   <xacro:include filename="$(find depthai_descriptions)/urdf/include/depthai_macro.urdf.xacro"/>
-  <xacro:macro name="piper_mount_oak_d_sr_handeye" params="parent_link simulation:=false oak_gazebo_rgbd_sensor:=false">
+  <!--
+    oak_visual_mesh=false: same TF tree as depthai OAK-D-SR but skip STL mesh on oak_model_origin (lighter RViz/MoveIt).
+    Defaults true for Gazebo / users who want the visual housing.
+  -->
+  <xacro:macro name="piper_mount_oak_d_sr_handeye" params="parent_link simulation:=false oak_gazebo_rgbd_sensor:=false oak_visual_mesh:=true">
     <link name="oak-d-base-frame"/>
     <joint name="piper_hand_eye_link6_mount" type="fixed">
       <origin
-        xyz="-0.068133439 0.007721162 0.055194547"
-        rpy="0.17430916 -1.23276438 -0.22762161"/>
+        xyz="-0.090866253 0.008472480 0.063306116"
+        rpy="0.030685051 -1.217622058 -0.102237087"/>
       <parent link="${parent_link}" />
       <child link="oak-d-base-frame" />
     </joint>
+    <xacro:if value="${oak_visual_mesh}">
     <xacro:depthai_camera
       camera_name="oak"
@@ -38,4 +46,40 @@
       simulation="${simulation}"
       rs_compat="false"/>
+    </xacro:if>
+    <!-- Mirrors depthai base_macro + OAK-D-SR stereo branch; omits oak_model_origin mesh link -->
+    <xacro:unless value="${oak_visual_mesh}">
+      <xacro:property name="oak_sr_pi" value="3.1415926535897931"/>
+      <xacro:property name="oak_sr_half_base" value="0.01"/>
+      <link name="oak-d_frame"/>
+      <joint name="oak_center_joint" type="fixed">
+        <parent link="oak-d-base-frame"/>
+        <child link="oak-d_frame"/>
+        <origin xyz="0 0 0" rpy="0 0 0"/>
+      </joint>
+      <link name="oak_left_camera_frame"/>
+      <joint name="oak_left_camera_joint" type="fixed">
+        <parent link="oak-d_frame"/>
+        <child link="oak_left_camera_frame"/>
+        <origin xyz="0 ${oak_sr_half_base} 0" rpy="0 0 0"/>
+      </joint>
+      <link name="oak_left_camera_optical_frame"/>
+      <joint name="oak_left_camera_optical_joint" type="fixed">
+        <origin xyz="0 0 0" rpy="-${oak_sr_pi/2} 0 -${oak_sr_pi/2}"/>
+        <parent link="oak_left_camera_frame"/>
+        <child link="oak_left_camera_optical_frame"/>
+      </joint>
+      <link name="oak_right_camera_frame"/>
+      <joint name="oak_right_camera_joint" type="fixed">
+        <parent link="oak-d_frame"/>
+        <child link="oak_right_camera_frame"/>
+        <origin xyz="0 -${oak_sr_half_base} 0" rpy="0 0 0"/>
+      </joint>
+      <link name="oak_right_camera_optical_frame"/>
+      <joint name="oak_right_camera_optical_joint" type="fixed">
+        <origin xyz="0 0 0" rpy="-${oak_sr_pi/2} 0 -${oak_sr_pi/2}"/>
+        <parent link="oak_right_camera_frame"/>
+        <child link="oak_right_camera_optical_frame"/>
+      </joint>
+    </xacro:unless>
     <xacro:if value="${oak_gazebo_rgbd_sensor}">
     <gazebo reference="oak_right_camera_frame">

File: src/robot_description/piper_description/urdf/piper_description.urdf (robot description, URDF)
Before this commit: robot piper, 10 links, 9 joints
Links:
- added link arm_tcp, mass 0.001
Joints:
- added joint arm_tcp_joint: type fixed, parent gripper_base, child arm_tcp, origin xyz=0 0 0.2411 rpy=0 0 0

File: src/robot_description/piper_description/urdf/piper_description.xacro (robot description, xacro)
@@ -3,5 +3,5 @@
   name="piper"
   xmlns:xacro="http://ros.org/wiki/xacro">
-  <xacro:include filename="$(find piper_description)/urdf/include/piper_oak_d_sr_handeye_macros.xacro"/>
+  <xacro:include filename="$(find piper_description)/urdf/include/piper_oak_d_pro_w_handeye_macros.xacro"/>
 <!-- world -->
   <link name="world"/>
@@ -338,5 +338,5 @@
       velocity="3" />
   </joint>
-  <xacro:piper_mount_oak_d_sr_handeye parent_link="link6" simulation="false" oak_gazebo_rgbd_sensor="false"/>
+  <xacro:piper_mount_oak_d_pro_w_handeye parent_link="link6" simulation="false" oak_visual_mesh="false"/>
   <link
     name="gripper_base">
@@ -505,4 +505,18 @@
       effort="10"
       velocity="1" />
+  </joint>
+  <!-- MoveIt / arm_api2 TCP: tool tip offset from gripper_base (+Z), 241.1 mm. -->
+  <xacro:property name="arm_tcp_xyz" value="0 0 0.2411"/>
+  <link name="arm_tcp">
+    <inertial>
+      <origin xyz="0 0 0" rpy="0 0 0" />
+      <mass value="0.001" />
+      <inertia ixx="1e-9" ixy="0" ixz="0" iyy="1e-9" iyz="0" izz="1e-9" />
+    </inertial>
+  </link>
+  <joint name="arm_tcp_joint" type="fixed">
+    <origin xyz="${arm_tcp_xyz}" rpy="0 0 0" />
+    <parent link="gripper_base" />
+    <child link="arm_tcp" />
   </joint>
 <!-- controller -->

File: src/robot_description/piper_description/urdf/piper_description_gazebo.xacro (robot description, xacro)
@@ -503,4 +503,18 @@
       effort="10"
       velocity="1" />
+  </joint>
+  <!-- MoveIt / arm_api2 TCP: tool tip offset from gripper_base (+Z), 241.1 mm. -->
+  <xacro:property name="arm_tcp_xyz" value="0 0 0.2411"/>
+  <link name="arm_tcp">
+    <inertial>
+      <origin xyz="0 0 0" rpy="0 0 0" />
+      <mass value="0.001" />
+      <inertia ixx="1e-9" ixy="0" ixz="0" iyy="1e-9" iyz="0" izz="1e-9" />
+    </inertial>
+  </link>
+  <joint name="arm_tcp_joint" type="fixed">
+    <origin xyz="${arm_tcp_xyz}" rpy="0 0 0" />
+    <parent link="gripper_base" />
+    <child link="arm_tcp" />
   </joint>
   <!-- Camera -->

File: src/robot_description/piper_description/urdf/piper_description_gz.xacro (robot description, xacro)
@@ -530,4 +530,18 @@
       friction="0" />
   </joint>
+  <!-- MoveIt / arm_api2 TCP: tool tip offset from gripper_base (+Z), 241.1 mm. -->
+  <xacro:property name="arm_tcp_xyz" value="0 0 0.2411"/>
+  <link name="arm_tcp">
+    <inertial>
+      <origin xyz="0 0 0" rpy="0 0 0" />
+      <mass value="0.001" />
+      <inertia ixx="1e-9" ixy="0" ixz="0" iyy="1e-9" iyz="0" izz="1e-9" />
+    </inertial>
+  </link>
+  <joint name="arm_tcp_joint" type="fixed">
+    <origin xyz="${arm_tcp_xyz}" rpy="0 0 0" />
+    <parent link="gripper_base" />
+    <child link="arm_tcp" />
+  </joint>
   <gazebo reference="base_link">
       <selfCollide>false</selfCollide>
