Commit message: feat: update OAK-D Pro W hand-eye mount and real gripper controller
Apply 2026-07-06 ChArUco calibration to link6→oak_rgb mount, switch URDF
to OAK-D-PRO-W with visual mesh, and drop joint8 from gripper_controller
so activation works on real hardware.

File: src/robot_description/piper_description/urdf/include/piper_oak_d_pro_w_handeye_macros.xacro (robot description, xacro)
@@ -2,13 +2,24 @@
 <!--
   Piper + OAK-D-PRO / OAK-D-PRO-W (depthai_ros_driver_v3 uses OAK-D-PRO URDF frames).
-  Calibration: eye-in-hand link6 → oak_rgb_camera_optical_frame.
-  Hand-eye estimate (link6→oak_rgb_camera_optical_frame): tx ty tz qx qy qz qw =
-    -0.0949 -0.0015 0.0437 -0.1250 0.1250 -0.6926 0.6993
-  link6 → oak-d-base-frame (REP-103 URDF roll-pitch-yaw = intrinsic XYZ):
-    xyz = -0.094900000 -0.001500000 0.043700000
-    rpy = 0.004813527 -1.215368884 0.004813527
+  Calibration: eye-in-hand link6 → oak_rgb_camera_optical_frame (ChArUco 13x9 board,
+  2026-07-06, 15 samples, residuals mean 6.5 mm / 1.4 deg).
+  Source: ~/.ros/hand_eye_calibration.yaml:
+    tracking_base_frame: oak_rgb_camera_optical_frame
+    robot_effector_frame: link6
+    tx ty tz qx qy qz qw =
+      -0.0936 0.0025 0.0443 0.1211 -0.1264 0.7035 -0.6888
+  The grasping point cloud is published in oak_rgb_camera_optical_frame — the same
+  frame this calibration targets. The mount origin below is solved as
+  T_mount = T_cal @ inv(T_nom_rgb) from depthai_descriptions_v3 nominal geometry,
+  so the stereo frames follow the camera's rigid internal layout (75 mm baseline).
   Do not run depthai driver with i_publish_tf_from_calibration or publish_description when
   using this macro — Piper robot_state_publisher owns the camera TF tree.
   Re-calibrate with hand_eye_calibration when the physical camera or mount changes.
+  After saving a new calibration from the GUI, regenerate the mount origin below with:
+    python3 -m hand_eye_calibration.depthai_mount_cli [dash]update-xacro path/to/this/file.xacro
+  (XML comments cannot contain a double dash: replace [dash] with two hyphens.)
+  (run from arms_ws/src/ros2_handeye_calibration; reads ~/.ros/hand_eye_calibration.yaml,
+  infers the rgb/right/left socket from tracking_base_frame). Then rebuild
+  piper_description and restart the robot stack.
 -->
 <robot xmlns:xacro="http://ros.org/wiki/xacro" name="piper_oak_d_pro_w_attachment_defs">
@@ -17,6 +28,6 @@
     <joint name="piper_hand_eye_link6_mount" type="fixed">
       <origin
-        xyz="-0.094900000 -0.001500000 0.043700000"
-        rpy="0.004813527 -1.215368884 0.004813527"/>
+        xyz="-0.093570378136 0.002501953147 0.044282542398"
+        rpy="0.010834909692 -1.219008031786 -0.032043316431"/>
       <parent link="${parent_link}"/>
       <child link="oak-d-base-frame"/>
@@ -27,5 +38,5 @@
         camera_name="oak"
         parent="oak-d-base-frame"
-        camera_model="OAK-D-PRO"
+        camera_model="OAK-D-PRO-W"
         base_frame="oak-d_frame"
         cam_pos_x="0.0"
@@ -42,5 +53,15 @@
       <xacro:property name="oak_pro_pi" value="3.1415926535897931"/>
       <xacro:property name="oak_pro_baseline" value="0.075"/>
-      <link name="oak-d_frame"/>
+      <link name="oak-d_frame">
+        <visual>
+          <origin xyz="0 0 0" rpy="0 0 0"/>
+          <geometry>
+            <box size="0.080 0.105 0.030"/>
+          </geometry>
+          <material name="oak_visual_black">
+            <color rgba="0.05 0.05 0.05 1.0"/>
+          </material>
+        </visual>
+      </link>
       <joint name="oak_center_joint" type="fixed">
         <parent link="oak-d-base-frame"/>

File: src/robot_description/piper_description/urdf/piper_description.xacro (robot description, xacro)
@@ -338,5 +338,5 @@
       velocity="3" />
   </joint>
-  <xacro:piper_mount_oak_d_pro_w_handeye parent_link="link6" simulation="false" oak_visual_mesh="false"/>
+  <xacro:piper_mount_oak_d_pro_w_handeye parent_link="link6" simulation="false" oak_visual_mesh="true"/>
   <link
     name="gripper_base">

Commit message: feat: add Femto Bolt hand-eye mount and welding-gun MoveIt config
Update the welding-gun URDF and demo launch, and add the Femto Bolt hand-eye macro plus an explicit OMPL planning config.

File: src/robot_description/piper_description/urdf/include/piper_oak_d_pro_w_handeye_macros.xacro (robot description, xacro)
@@ -19,5 +19,5 @@
     python3 -m hand_eye_calibration.depthai_mount_cli [dash]update-xacro path/to/this/file.xacro
   (XML comments cannot contain a double dash: replace [dash] with two hyphens.)
-  (run from arms_ws/src/ros2_handeye_calibration; reads ~/.ros/hand_eye_calibration.yaml,
+  (run from arms_ws/src/misc/ros2_handeye_calibration; reads ~/.ros/hand_eye_calibration.yaml,
   infers the rgb/right/left socket from tracking_base_frame). Then rebuild
   piper_description and restart the robot stack.

File: src/robot_description/piper_description/urdf/piper_welding_gun.urdf.xacro (robot description, xacro)
@@ -26,18 +26,37 @@
     <origin xyz="0 0 0" rpy="0 0 0"/>
   </joint>
-  <!-- CAD tip face centre; bent nozzle axis is (sin(35deg),0,cos(35deg)).
-       Keep arm_tcp as the shared MoveIt/arm_api2 endpoint; TCP +X follows wire. -->
+  <!-- TCP pivot/axis calibration 2026-09-23T14:02:51Z, parent link6.
+       Calibrated +Z is expressed as arm_tcp +X for the welding planner.
+       Position RMS 3.54 mm; independent physical validation is still required.
+       The gun mount is identity, so the flange-relative origin applies here. -->
   <link name="arm_tcp"/>
   <joint name="arm_tcp_joint" type="fixed">
     <parent link="piper_welding_gun"/><child link="arm_tcp"/>
-    <origin xyz="0.05360585785 0 0.2085160675" rpy="0 -0.9599310886 0"/>
+    <!-- Simulation: tip of the CAD wire/contact tip (end of the 3 mm stub), on the
+         35 deg bent nozzle axis (sin 35, 0, cos 35); TCP +X follows the wire. The
+         real robot keeps the calibrated pivot, which is not on the CAD axis. -->
+    <xacro:if value="$(arg simulation)">
+      <origin xyz="0.05360585785 0 0.2085160675" rpy="0 -0.9599310886 0"/>
+    </xacro:if>
+    <xacro:unless value="$(arg simulation)">
+      <origin xyz="0.059716507277 -0.002810430194 0.190158035855" rpy="-0.027929237913 -0.909524738174 0.022044250167"/>
+    </xacro:unless>
   </joint>
-  <xacro:include filename="$(find piper_description)/urdf/include/piper_realsense_d435_handeye_macros.xacro"/>
-  <xacro:piper_mount_realsense_d435_handeye parent_link="link6"/>
+  <xacro:if value="${'$(arg wrist_camera)' == 'femto_bolt'}">
+    <xacro:include filename="$(find piper_description)/urdf/include/piper_femto_bolt_handeye_macros.xacro"/>
+    <xacro:piper_mount_femto_bolt_handeye parent_link="link6" use_nominal_extrinsics="$(arg simulation)"/>
+  </xacro:if>
+  <xacro:unless value="${'$(arg wrist_camera)' == 'femto_bolt'}">
+    <xacro:include filename="$(find piper_description)/urdf/include/piper_realsense_d435_handeye_macros.xacro"/>
+    <xacro:piper_mount_realsense_d435_handeye parent_link="link6"/>
+  </xacro:unless>
   <!-- Preserve the existing simulated-camera topic/frame API used by the GUI. -->
+  <!-- Driver-owned Femto optical frames are not links in the real URDF. -->
+  <xacro:if value="${'$(arg simulation)' == 'true' or '$(arg wrist_camera)' != 'femto_bolt'}">
   <link name="oak_right_camera_optical_frame"/>
   <joint name="piper_sim_optical_alias" type="fixed">
     <parent link="camera_color_optical_frame"/><child link="oak_right_camera_optical_frame"/>
   </joint>
+  </xacro:if>
   <xacro:if value="$(arg simulation)">
   <xacro:include filename="$(find piper_description)/urdf/include/d435_gazebo_sensors.xacro"/>
