Commit message: feat: use pivot-calibrated welding gun TCP and link5 Femto mount in simulation
Real robot gets TCP-v6-pivot, simulation keeps the model wire tip. The
simulated Femto now sits on link5 with the HE-v8 optical pose, and the
flange collisions are disabled in the sim SRDF.

Co-Authored-By: Claude Opus 5.5 <noreply@anthropic.com>

File: src/robot_description/piper_description/urdf/include/piper_femto_bolt_handeye_macros.xacro (robot description, xacro)
@@ -1,7 +1,8 @@
 <?xml version="1.0"?>
 <!--
-  Piper + Orbbec Femto Bolt (eye-in-hand; real mount on link5 since 2026-10-05,
-  simulation on link6). The real origin below is relative to that parent link and
-  is stale until the new mount is calibrated (robot_effector_frame:=link5).
+  Piper + Orbbec Femto Bolt (eye-in-hand; mount on link5 since 2026-10-05, real
+  and simulation). Real origin = HE-v8-link5. The simulation (nominal) origin is
+  the same HE-v8 link5 -> camera_color_optical_frame pose re-expressed through the
+  nominal internal camera chain, so the simulated optical frame matches the real one.
   Frame names match orbbec_camera's femto_bolt.launch.py defaults (camera_name:=camera):
     camera_base_link, camera_link, camera_color_optical_frame, etc.
@@ -24,9 +25,9 @@
     <xacro:include filename="$(find orbbec_description)/urdf/femto_bolt.urdf.xacro"/>
     <xacro:femto_bolt prefix="camera" parent="${parent_link}" use_nominal_extrinsics="${use_nominal_extrinsics}">
-      <!-- Preserve the original nominal-chain hand-eye optical pose. The real
+      <!-- Nominal: HE-v8-link5 optical pose through the nominal chain. The real
            mount is re-expressed using this camera's recorded driver extrinsics
            (2026-09-24); internal TFs themselves always come from the driver. -->
-      <origin xyz="${'-0.116960119269 0.004378100746 -0.028825832440' if use_nominal_extrinsics else '-0.044525749544 -0.064654994020 -0.003299954006'}"
-              rpy="${'0.062955579669 -0.945517293938 -0.083284514853' if use_nominal_extrinsics else '1.698973335600 -0.016012269413 -1.559219138477'}"/>
+      <origin xyz="${'-0.044371623019 -0.064359369068 -0.002761697893' if use_nominal_extrinsics else '-0.044525749544 -0.064654994020 -0.003299954006'}"
+              rpy="${'1.698960611174 -0.015341477877 -1.559133329065' if use_nominal_extrinsics else '1.698973335600 -0.016012269413 -1.559219138477'}"/>
     </xacro:femto_bolt>
   </xacro:macro>

File: src/robot_description/piper_description/urdf/piper_welding_gun.urdf.xacro (robot description, xacro)
@@ -64,10 +64,17 @@
     <!-- Wire tip of 03_welding_gun.stl on the AgileX flange (model geometry, 2026-10-05):
          end-face centre of the Ø3 mm wire, axis 45.3 deg from link6 Z toward +X.
-         TCP +X follows the wire. Same for real robot and simulation. -->
-    <origin xyz="0.039746665881 -0.000003287520 0.111796185844" rpy="0 -0.7801056516 0"/>
+         TCP +X follows the wire. Simulation keeps this model tip. -->
+    <xacro:if value="$(arg simulation)">
+      <origin xyz="0.039746665881 -0.000003287520 0.111796185844" rpy="0 -0.7801056516 0"/>
+    </xacro:if>
+    <!-- Real robot: TCP-v6-pivot (2026-10-06). Wire tip from the spike pivot calibration
+         (Tool TCP GUI, no camera) - 8 mm along the wire (TCP +X) on request (2026-10-06). Model wire direction kept. -->
+    <xacro:unless value="$(arg simulation)">
+      <origin xyz="0.03401 -0.0003 0.10577" rpy="0 -0.7801056516 0"/>
+    </xacro:unless>
   </joint>
   <xacro:if value="${'$(arg wrist_camera)' == 'femto_bolt'}">
     <xacro:include filename="$(find piper_description)/urdf/include/piper_femto_bolt_handeye_macros.xacro"/>
-    <xacro:piper_mount_femto_bolt_handeye parent_link="${'link6' if '$(arg simulation)' == 'true' else '$(arg femto_parent_link)'}"
+    <xacro:piper_mount_femto_bolt_handeye parent_link="$(arg femto_parent_link)"
                                          use_nominal_extrinsics="$(arg simulation)"/>
   </xacro:if>

Commit message: feat(piper_description): load welding-gun Femto mount and TCP from calibration YAML
piper_femto_bolt_handeye_macros.xacro and arm_tcp_joint in
piper_welding_gun.urdf.xacro no longer hold calibration values: they
xacro.load_yaml the files given by the femto_calibration / tcp_calibration
args (real + nominal/sim origins). Defaults in config/calibration/ keep the
previous values (HE-v8-link5, TCP-v6, gun model tip); generated URDF is
identical.

piper_sim_moveit.launch.py and demo_welding_gun_realsense.launch.py pass the
robot's active ~/.ros/calibration/<robot_id>/<mount>/current.yaml (else the
default), and run move_group with respawn and without a robot_description
parameter (it reads robot_state_publisher's topic), so GUI Apply can restart
only move_group. Real launch: publish_robot_description off.

Co-Authored-By: Claude Opus 5.5 <noreply@anthropic.com>

File: src/robot_description/piper_description/urdf/include/piper_femto_bolt_handeye_macros.xacro (robot description, xacro)
@@ -2,7 +2,14 @@
 <!--
   Piper + Orbbec Femto Bolt (eye-in-hand; mount on link5 since 2026-10-05, real
-  and simulation). Real origin = HE-v8-link5. The simulation (nominal) origin is
-  the same HE-v8 link5 -> camera_color_optical_frame pose re-expressed through the
-  nominal internal camera chain, so the simulated optical frame matches the real one.
+  and simulation).
+  The mount origin (parent_link -> camera_base_link) is NOT written here. It is
+  loaded from calibration_file, a YAML with a `real` and a `nominal` origin:
+    - normally the robot's active calibration
+      ~/.ros/calibration/<robot_id>/femto_bolt_handeye/current.yaml, written by
+      GUI Apply / handeye_welding_gun_apply (hand_eye_calibration/calibration_store.py);
+    - otherwise piper_description/config/calibration/femto_bolt_handeye_default.yaml.
+  Real: the optical pose re-expressed through the driver's own depth->colour
+  extrinsics. Nominal (simulation): the same optical pose through the nominal
+  chain of orbbec_description's femto_bolt macro, so both optical frames match.
   Frame names match orbbec_camera's femto_bolt.launch.py defaults (camera_name:=camera):
     camera_base_link, camera_link, camera_color_optical_frame, etc.
@@ -10,24 +17,12 @@
   The Orbbec driver owns all internal camera TFs (publish_tf:=true).
   Simulation uses nominal internal transforms because no camera driver runs.
-  Calibration: eye-in-hand link6 -> camera_color_optical_frame from arm_api2 GUI
-  hand-eye calibration (2026-09-23 14:37 UTC; 15 samples, 13 inliers,
-  Daniilidis + nonlinear refinement; 2.57mm / 0.94deg mean residual,
-  3.25mm worst-direction 1-sigma uncertainty; not
-  independently validated). The origin below is converted from that
-  optical-frame estimate to the Femto Bolt's own bottom-mount base_link frame
-  used by orbbec_description's femto_bolt xacro macro (base_link -> link ->
-  depth_frame -> color_frame -> color_optical_frame fixed offsets baked into
-  that macro). Re-calibrate with hand_eye_calibration and update the fixed
-  joint origin when the physical mount or camera changes.
 -->
 <robot xmlns:xacro="http://ros.org/wiki/xacro" name="piper_femto_bolt_attachment_defs">
-  <xacro:macro name="piper_mount_femto_bolt_handeye" params="parent_link use_nominal_extrinsics:=false">
+  <xacro:macro name="piper_mount_femto_bolt_handeye" params="parent_link calibration_file use_nominal_extrinsics:=false">
+    <xacro:property name="femto_cal" value="${xacro.load_yaml(calibration_file)}"/>
+    <xacro:property name="femto_origin" value="${femto_cal['nominal'] if use_nominal_extrinsics else femto_cal['real']}"/>
     <xacro:include filename="$(find orbbec_description)/urdf/femto_bolt.urdf.xacro"/>
     <xacro:femto_bolt prefix="camera" parent="${parent_link}" use_nominal_extrinsics="${use_nominal_extrinsics}">
-      <!-- Nominal: HE-v8-link5 optical pose through the nominal chain. The real
-           mount is re-expressed using this camera's recorded driver extrinsics
-           (2026-09-24); internal TFs themselves always come from the driver. -->
-      <origin xyz="${'-0.044371623019 -0.064359369068 -0.002761697893' if use_nominal_extrinsics else '-0.044525749544 -0.064654994020 -0.003299954006'}"
-              rpy="${'1.698960611174 -0.015341477877 -1.559133329065' if use_nominal_extrinsics else '1.698973335600 -0.016012269413 -1.559219138477'}"/>
+      <origin xyz="${femto_origin['xyz']}" rpy="${femto_origin['rpy']}"/>
     </xacro:femto_bolt>
   </xacro:macro>

File: src/robot_description/piper_description/urdf/piper_welding_gun.urdf.xacro (robot description, xacro)
@@ -7,4 +7,9 @@
        Simulation keeps link6 because its nominal extrinsics are expressed there. -->
   <xacro:arg name="femto_parent_link" default="link5"/>
+  <!-- Femto mount calibration (real + nominal origin). Launch files pass the robot's
+       active ~/.ros/calibration/<robot_id>/femto_bolt_handeye/current.yaml; the repo
+       default only applies when that does not exist (calibration_store.py). -->
+  <xacro:arg name="femto_calibration" default="$(find piper_description)/config/calibration/femto_bolt_handeye_default.yaml"/>
+  <xacro:arg name="tcp_calibration" default="$(find piper_description)/config/calibration/welding_gun_tcp_default.yaml"/>
   <xacro:include filename="$(find piper_description)/urdf/piper_no_gripper_description_gz.xacro"/>
   <!-- AgileX PiPER flange (STL in mm): mounting face on link6 at Z=0, top recess Ø40.5 x 6 mm. -->
@@ -60,22 +65,19 @@
   <!-- Nominal CAD wire-tip TCP, applied 2026-09-30. TCP +X follows the wire. -->
   <link name="arm_tcp"/>
+  <!-- Welding-gun TCP (real + sim origin). Launch files pass the robot's active
+       ~/.ros/calibration/<robot_id>/welding_gun_tcp/current.yaml; the repo default
+       (config/calibration/welding_gun_tcp_default.yaml) applies when that does not exist.
+       TCP +X follows the wire. -->
+  <xacro:property name="tcp_cal" value="${xacro.load_yaml('$(arg tcp_calibration)')}"/>
+  <xacro:property name="tcp_origin" value="${tcp_cal['sim'] if '$(arg simulation)' == 'true' else tcp_cal['real']}"/>
   <joint name="arm_tcp_joint" type="fixed">
     <parent link="piper_welding_gun"/><child link="arm_tcp"/>
-    <!-- Wire tip of 03_welding_gun.stl on the AgileX flange (model geometry, 2026-10-05):
-         end-face centre of the Ø3 mm wire, axis 45.3 deg from link6 Z toward +X.
-         TCP +X follows the wire. Simulation keeps this model tip. -->
-    <xacro:if value="$(arg simulation)">
-      <origin xyz="0.039746665881 -0.000003287520 0.111796185844" rpy="0 -0.7801056516 0"/>
-    </xacro:if>
-    <!-- Real robot: TCP-v6-pivot (2026-10-06). Wire tip from the spike pivot calibration
-         (Tool TCP GUI, no camera) - 8 mm along the wire (TCP +X) on request (2026-10-06). Model wire direction kept. -->
-    <xacro:unless value="$(arg simulation)">
-      <origin xyz="0.03401 -0.0003 0.10577" rpy="0 -0.7801056516 0"/>
-    </xacro:unless>
+    <origin xyz="${tcp_origin['xyz']}" rpy="${tcp_origin['rpy']}"/>
   </joint>
   <xacro:if value="${'$(arg wrist_camera)' == 'femto_bolt'}">
     <xacro:include filename="$(find piper_description)/urdf/include/piper_femto_bolt_handeye_macros.xacro"/>
     <xacro:piper_mount_femto_bolt_handeye parent_link="$(arg femto_parent_link)"
-                                         use_nominal_extrinsics="$(arg simulation)"/>
+                                         use_nominal_extrinsics="$(arg simulation)"
+                                         calibration_file="$(arg femto_calibration)"/>
   </xacro:if>
   <xacro:unless value="${'$(arg wrist_camera)' == 'femto_bolt'}">
