Commit message: feat: add welding-gun URDF/MoveIt config and D435 Gazebo simulation
Co-authored-by: Cursor <cursoragent@cursor.com>

File: src/robot_description/piper_description/urdf/include/piper_realsense_d435_handeye_macros.xacro (robot description, xacro)
@@ -7,5 +7,5 @@
   robot_state_publisher owns the camera TF tree (same pattern as OAK-D Pro W).
   Calibration: eye-in-hand link6 → camera_color_optical_frame from arm_api2 GUI
-  hand-eye calibration (2026-07-14). The origin below is converted from that
+  hand-eye calibration (2026-09-14). The origin below is converted from that
   optical-frame estimate to the D435 bottom screw frame used by sensor_d435.
   Re-calibrate with hand_eye_calibration and update the fixed joint origin when
@@ -21,6 +21,6 @@
       add_plug="false"
       use_mesh="${use_mesh}">
-      <origin xyz="-0.085175061982 0.003246095153 0.029951767255"
-              rpy="-0.025292882305 -1.208671109768 0.020260903849"/>
+      <origin xyz="-0.075244452946 0.003546591618 0.047111111066"
+              rpy="-0.004648673805 -1.226424370880 0.006596038054"/>
     </xacro:sensor_d435>
   </xacro:macro>

File: src/robot_description/piper_description/urdf/piper_no_gripper_description_gz.xacro (robot description, xacro)
@@ -3,5 +3,9 @@
   name="piper"
   xmlns:xacro="http://ros.org/wiki/xacro">
+<xacro:arg name="simulation" default="true"/>
+<xacro:arg name="wrist_camera" default="gazebo_oak"/>
 <!-- world -->
+  <!-- Finishes estimated from https://global.agilex.ai/products/piper:
+       black joint housings/base, graphite arms, metallic tool flange. -->
   <link name="world"/>
   <joint name="fixed_base_joint" type="fixed">
@@ -25,8 +29,7 @@
           filename="file://$(find piper_description)/meshes/base_link.STL" />
       </geometry>
-      <material
-        name="">
-        <color
-          rgba="0.792156862745098 0.819607843137255 0.933333333333333 1" />
+      <material name="piper_base_link_finish">
+        <color
+          rgba="0.055 0.055 0.055 1" />
       </material>
     </visual>
@@ -56,8 +59,7 @@
           filename="file://$(find piper_description)/meshes/link1.STL" />
       </geometry>
-      <material
-        name="">
-        <color
-          rgba="0.792156862745098 0.819607843137255 0.933333333333333 1" />
+      <material name="piper_link1_finish">
+        <color
+          rgba="0.055 0.055 0.055 1" />
       </material>
     </visual>
@@ -105,8 +107,7 @@
           filename="file://$(find piper_description)/meshes/link2.STL" />
       </geometry>
-      <material
-        name="">
-        <color
-          rgba="0.792156862745098 0.819607843137255 0.933333333333333 1" />
+      <material name="piper_link2_finish">
+        <color
+          rgba="0.28 0.28 0.28 1" />
       </material>
     </visual>
@@ -154,8 +155,7 @@
           filename="file://$(find piper_description)/meshes/link3.STL" />
       </geometry>
-      <material
-        name="">
-        <color
-          rgba="0.792156862745098 0.819607843137255 0.933333333333333 1" />
+      <material name="piper_link3_finish">
+        <color
+          rgba="0.28 0.28 0.28 1" />
       </material>
     </visual>
@@ -203,8 +203,7 @@
           filename="file://$(find piper_description)/meshes/link4.STL" />
       </geometry>
-      <material
-        name="">
-        <color
-          rgba="0.792156862745098 0.819607843137255 0.933333333333333 1" />
+      <material name="piper_link4_finish">
+        <color
+          rgba="0.055 0.055 0.055 1" />
       </material>
     </visual>
@@ -252,8 +251,7 @@
           filename="file://$(find piper_description)/meshes/link5.STL" />
       </geometry>
-      <material
-        name="">
-        <color
-          rgba="0.792156862745098 0.819607843137255 0.933333333333333 1" />
+      <material name="piper_link5_finish">
+        <color
+          rgba="0.055 0.055 0.055 1" />
       </material>
     </visual>
@@ -301,8 +299,7 @@
           filename="file://$(find piper_description)/meshes/link6.STL" />
       </geometry>
-      <material
-        name="">
-        <color
-          rgba="0.898039215686275 0.917647058823529 0.929411764705882 1" />
+      <material name="piper_link6_finish">
+        <color
+          rgba="0.5 0.5 0.5 1" />
       </material>
     </visual>
@@ -336,5 +333,9 @@
   </joint>
   <xacro:include filename="$(find piper_description)/urdf/include/piper_oak_d_sr_handeye_macros.xacro"/>
-  <xacro:piper_mount_oak_d_sr_handeye parent_link="link6" simulation="true" oak_gazebo_rgbd_sensor="true" oak_visual_mesh="false"/>
+  <xacro:property name="no_gripper_camera" value="$(arg wrist_camera)"/>
+  <xacro:if value="${no_gripper_camera == 'gazebo_oak'}">
+    <xacro:piper_mount_oak_d_sr_handeye parent_link="link6" simulation="true" oak_gazebo_rgbd_sensor="true" oak_visual_mesh="false"/>
+  </xacro:if>
+  <xacro:if value="$(arg simulation)">
   <gazebo reference="base_link">
       <selfCollide>false</selfCollide>
@@ -447,3 +448,4 @@
       </joint>
   </ros2_control>
+  </xacro:if>
 </robot>

Commit message: fix: update D435 hand-eye extrinsics from latest calibration
Replace the previous mount origin with the measured transform so RealSense optical frame matches the current Piper eye-in-hand setup.

Co-authored-by: Cursor <cursoragent@cursor.com>

File: src/robot_description/piper_description/urdf/include/piper_realsense_d435_handeye_macros.xacro (robot description, xacro)
@@ -21,6 +21,5 @@
       add_plug="false"
       use_mesh="${use_mesh}">
-      <origin xyz="-0.075244452946 0.003546591618 0.047111111066"
-              rpy="-0.004648673805 -1.226424370880 0.006596038054"/>
+      <origin xyz="-0.081443840090 -0.001060325492 0.040086067573" rpy="-0.007029573507 -1.205748634070 -0.013835835278"/>
     </xacro:sensor_d435>
   </xacro:macro>

Commit message: fix(piper_description): apply calibrated D435 mount and joint zero offsets
- replace D435 hand-eye origin with the 2026-10-14 calibration result
- add joint2..5 zero offsets on the real robot only (simulation keeps nominal)
- set gripper xyz 5.8 mm in piper_no_gripper_description_gz.xacro
- add 1.048 mm flange-axis offset for the welding gun, real robot only

Co-Authored-By: Claude Opus 5.5 <noreply@anthropic.com>

File: src/robot_description/piper_description/urdf/include/piper_realsense_d435_handeye_macros.xacro (robot description, xacro)
@@ -7,6 +7,11 @@
   robot_state_publisher owns the camera TF tree (same pattern as OAK-D Pro W).
   Calibration: eye-in-hand link6 → camera_color_optical_frame from arm_api2 GUI
-  hand-eye calibration (2026-09-14). The origin below is converted from that
-  optical-frame estimate to the D435 bottom screw frame used by sensor_d435.
+  hand-eye calibration (2026-09-14); replaced 2026-10-13 by HE-v9-D435-Intrinsic-26
+  (run 20261013_095104, FORCED on user request: acceptance failed, position RMS 5.20 mm), then on
+  2026-10-14 by the camera_joint estimated together with the PiPER joint2..5 zero offsets
+  (robot_calibration, runs 20261013_090057/095104/145212, 70 views; link6 -> optical
+  -87.8/34.4/46.1 mm; diagnostics/piper_joint_offsets_20261013). This mount is only valid
+  with those offsets in piper_description.xacro. Previous origin (HE-v9):
+  xyz="-0.083398718061 -0.000596015924 0.008566408033" rpy="-0.031901801676 -1.216619402843 0.033971246659".
   Re-calibrate with hand_eye_calibration and update the fixed joint origin when
   the physical mount or camera changes.
@@ -21,5 +26,5 @@
       add_plug="false"
       use_mesh="${use_mesh}">
-      <origin xyz="-0.081443840090 -0.001060325492 0.040086067573" rpy="-0.007029573507 -1.205748634070 -0.013835835278"/>
+      <origin xyz="-0.07895832 0.00190165 0.03214706" rpy="-0.03568854 -1.20919161 0.06005394"/>
     </xacro:sensor_d435>
   </xacro:macro>

File: src/robot_description/piper_description/urdf/piper_description.xacro (robot description, xacro)
@@ -130,5 +130,6 @@
     <origin
       xyz="0 0 0"
-      rpy="1.5708 -0.1359 -3.1416" />
+      rpy="1.570800004 -0.144020257 3.141585277" />
+      <!-- Zero offset +0.465 deg from camera kinematic calibration 2026-10-13 (robot_calibration, 70 D435 views; diagnostics/piper_joint_offsets_20261013): origin = nominal * Rz(offset), nominal rpy="1.5708 -0.1359 -3.1416". Revert: diagnostics/piper_joint_offsets_20261013/apply_20261014/before_piper_description.xacro -->
       <!-- rpy="1.5708 -0.10095-0.03490659 -3.1416" /> -->
     <parent
@@ -180,5 +181,6 @@
     <origin
       xyz="0.28503 0 0"
-      rpy="0 0 -1.7939" />
+      rpy="0 0 -1.771126297" />
+      <!-- Zero offset +1.305 deg from camera kinematic calibration 2026-10-13 (robot_calibration, 70 D435 views; diagnostics/piper_joint_offsets_20261013): origin = nominal * Rz(offset), nominal rpy="0 0 -1.7939". Revert: diagnostics/piper_joint_offsets_20261013/apply_20261014/before_piper_description.xacro -->
       <!-- rpy="0 0 -1.759-0.03490659" /> -->
     <parent
@@ -230,5 +232,6 @@
     <origin
       xyz="-0.021984 -0.25075 0"
-      rpy="1.5708 0 0" />
+      rpy="1.5708 -0.008825978 -0.000000032" />
+      <!-- Zero offset +0.506 deg from camera kinematic calibration 2026-10-13 (robot_calibration, 70 D435 views; diagnostics/piper_joint_offsets_20261013): origin = nominal * Rz(offset), nominal rpy="1.5708 0 0". Revert: diagnostics/piper_joint_offsets_20261013/apply_20261014/before_piper_description.xacro -->
     <parent
       link="link3" />
@@ -279,5 +282,6 @@
     <origin
       xyz="0 0 0"
-      rpy="-1.5708 0 0" />
+      rpy="-1.5708 -0.007785459 0.000000029" />
+      <!-- Zero offset -0.446 deg from camera kinematic calibration 2026-10-13 (robot_calibration, 70 D435 views; diagnostics/piper_joint_offsets_20261013): origin = nominal * Rz(offset), nominal rpy="-1.5708 0 0". Revert: diagnostics/piper_joint_offsets_20261013/apply_20261014/before_piper_description.xacro -->
     <parent
       link="link4" />
@@ -391,6 +395,7 @@
     type="fixed">
     <origin
-      xyz="0 0 0"
+      xyz="0 0 0.0058"
       rpy="0 0 0" />
+    <!-- Gripper 5.8 mm further along the flange axis than the official model (mounting spacer/bracket), 2026-10-14: set so the closed fingers resting on the table (2 cm below base_link, riser) meet it with the gripper pointing straight down; the ruler gave 145 mm flange -> tips (9.2 mm), which overshot by 3.4 mm. Was xyz="0 0 0". Gripper tilt is not modelled; refine with a Tool TCP pivot. -->
     <parent
       link="link6" />

File: src/robot_description/piper_description/urdf/piper_no_gripper_description_gz.xacro (robot description, xacro)
@@ -5,4 +5,19 @@
 <xacro:arg name="simulation" default="true"/>
 <xacro:arg name="wrist_camera" default="gazebo_oak"/>
+<!-- PiPER joint2..5 zero offsets (camera kinematic calibration 2026-10-13/14, robot_calibration, 70 D435 views;
+     diagnostics/piper_joint_offsets_20261013): origin = nominal * Rz(offset). Real robot only (simulation:=false);
+     Gazebo keeps the nominal origins. Same values as piper_description.xacro. -->
+<xacro:if value="$(arg simulation)">
+  <xacro:property name="joint2_origin_rpy" value="1.5708 -0.1359 -3.1416"/>
+  <xacro:property name="joint3_origin_rpy" value="0 0 -1.7939"/>
+  <xacro:property name="joint4_origin_rpy" value="1.5708 0 0"/>
+  <xacro:property name="joint5_origin_rpy" value="-1.5708 0 0"/>
+</xacro:if>
+<xacro:unless value="$(arg simulation)">
+  <xacro:property name="joint2_origin_rpy" value="1.570800004 -0.144020257 3.141585277"/>  <!-- +0.465 deg -->
+  <xacro:property name="joint3_origin_rpy" value="0 0 -1.771126297"/>  <!-- +1.305 deg -->
+  <xacro:property name="joint4_origin_rpy" value="1.5708 -0.008825978 -0.000000032"/>  <!-- +0.506 deg -->
+  <xacro:property name="joint5_origin_rpy" value="-1.5708 -0.007785459 0.000000029"/>  <!-- -0.446 deg -->
+</xacro:unless>
 <!-- world -->
   <!-- Finishes estimated from https://global.agilex.ai/products/piper:
@@ -127,5 +142,5 @@
     <origin
       xyz="0 0 0"
-      rpy="1.5708 -0.1359 -3.1416" />
+      rpy="${joint2_origin_rpy}" />
     <parent
       link="link1" />
@@ -175,5 +190,5 @@
     <origin
       xyz="0.28503 0 0"
-      rpy="0 0 -1.7939" />
+      rpy="${joint3_origin_rpy}" />
     <parent
       link="link2" />
@@ -223,5 +238,5 @@
     <origin
       xyz="-0.021984 -0.25075 0"
-      rpy="1.5708 0 0" />
+      rpy="${joint4_origin_rpy}" />
     <parent
       link="link3" />
@@ -271,5 +286,5 @@
     <origin
       xyz="0 0 0"
-      rpy="-1.5708 0 0" />
+      rpy="${joint5_origin_rpy}" />
     <parent
       link="link4" />

File: src/robot_description/piper_description/urdf/piper_welding_gun.urdf.xacro (robot description, xacro)
@@ -59,7 +59,11 @@
     </inertial>
   </link>
+  <!-- Real robot only: gun 1.048 mm further out along the flange axis (link6 z), so the
+       CAD wire tip touching the table reads z = -20.0 mm (base on a 2 cm plate); measured
+       2026-10-14 at joints (-0.009, 1.599, -0.002, 0.064, -0.733, 0). Simulation keeps the CAD mount. -->
+  <xacro:property name="gun_mount_z" value="${0.001048 if '$(arg simulation)' == 'false' else 0.0}"/>
   <joint name="piper_welding_gun_mount" type="fixed">
     <parent link="piper_flange"/><child link="piper_welding_gun"/>
-    <origin xyz="0 0 0" rpy="0 0 0"/>
+    <origin xyz="0 0 ${gun_mount_z}" rpy="0 0 0"/>
   </joint>
   <!-- Nominal CAD wire-tip TCP, applied 2026-09-30. TCP +X follows the wire. -->
