Commit message: feat: enhance hybrid OAK-D Pro W integration and simulation configurations
- Added joint limits for the OAK-D Pro W to ensure proper planning in Gazebo.
- Updated launch files to support hybrid mode with DepthAI driver and simulation time synchronization.
- Introduced new configuration files for hybrid operation and adjusted existing launch scripts for better flexibility.
- Included a new script for synchronizing timestamps between the real camera and Gazebo.
- Enhanced URDF and xacro files to accommodate different wrist camera configurations.

This commit improves the overall functionality and usability of the Piper simulation with the OAK-D Pro W camera.

File: src/piper_sim/piper_gazebo/urdf/piper_gz.urdf.xacro (robot description, xacro)
@@ -3,4 +3,6 @@
   <!-- Arguments -->
   <xacro:arg name="simulation_controllers" default="" />
+  <!-- gazebo_oak | oak_d_pro_w | none (hybrid: real OAK-D Pro W + stamp sync) -->
+  <xacro:arg name="wrist_camera" default="gazebo_oak" />
   <!-- Include Piper description -->
   <xacro:include filename="$(find piper_description)/urdf/piper_description_gz.xacro"/>
@@ -9,4 +11,6 @@
     <plugin filename="gz_ros2_control-system" name="gz_ros2_control::GazeboSimROS2ControlPlugin">
       <parameters>$(arg simulation_controllers)</parameters>
+      <hold_joints>true</hold_joints>
+      <position_proportional_gain>0.1</position_proportional_gain>
     </plugin>
   </gazebo>

File: src/piper_sim/piper_gazebo/urdf/piper_gz_no_gripper.urdf.xacro (robot description, xacro)
@@ -6,4 +6,6 @@
     <plugin filename="gz_ros2_control-system" name="gz_ros2_control::GazeboSimROS2ControlPlugin">
       <parameters>$(arg simulation_controllers)</parameters>
+      <hold_joints>true</hold_joints>
+      <position_proportional_gain>0.1</position_proportional_gain>
     </plugin>
   </gazebo>

File: src/robot_description/piper_description/urdf/piper_description_gz.xacro (robot description, xacro)
@@ -3,4 +3,6 @@
   name="piper"
   xmlns:xacro="http://ros.org/wiki/xacro">
+  <xacro:arg name="wrist_camera" default="gazebo_oak"/>
+  <xacro:property name="wrist_camera_selected" value="$(arg wrist_camera)"/>
 <!-- world -->
   <link name="world"/>
@@ -356,5 +358,12 @@
   </joint>
   <xacro:include filename="$(find piper_description)/urdf/include/piper_oak_d_sr_handeye_macros.xacro"/>
-  <xacro:piper_mount_oak_d_sr_handeye parent_link="link6" simulation="true" oak_gazebo_rgbd_sensor="true" oak_visual_mesh="false"/>
+  <xacro:include filename="$(find piper_description)/urdf/include/piper_oak_d_pro_w_handeye_macros.xacro"/>
+  <xacro:if value="${wrist_camera_selected == 'gazebo_oak'}">
+    <xacro:piper_mount_oak_d_sr_handeye parent_link="link6" simulation="true" oak_gazebo_rgbd_sensor="true" oak_visual_mesh="false"/>
+  </xacro:if>
+  <xacro:if value="${wrist_camera_selected == 'oak_d_pro_w'}">
+    <!-- Hybrid: calibrated Pro W TF tree, no Gazebo RGB-D sensor. -->
+    <xacro:piper_mount_oak_d_pro_w_handeye parent_link="link6" simulation="false" oak_visual_mesh="false"/>
+  </xacro:if>
   <link
     name="gripper_base">
