Commit message: feat: add piper_hardware ros2_control system and welding gun model
Add SDK backend, CAN feedback and command guard for the Piper driver,
a piper_hardware ros2_control plugin with tests, welding gun and flange
meshes, a ChArUco 6x8 Gazebo model, and updated MoveIt configs.

Co-Authored-By: Claude Opus 5.5 <noreply@anthropic.com>

File: src/piper_moveit/piper_no_gripper_moveit/config/piper.ros2_control.xacro (robot description, xacro)
@@ -1,10 +1,19 @@
 <?xml version="1.0"?>
 <robot xmlns:xacro="http://www.ros.org/wiki/xacro">
-    <xacro:macro name="piper_ros2_control" params="name initial_positions_file">
+    <xacro:macro name="piper_ros2_control" params="name initial_positions_file use_mock_hardware:=false">
         <xacro:property name="initial_positions" value="${load_yaml(initial_positions_file)['initial_positions']}"/>
         <ros2_control name="${name}" type="system">
             <hardware>
-                <!-- By default, set up controllers for simulation. This won't work on real hardware -->
-                <plugin>mock_components/GenericSystem</plugin>
+                <xacro:if value="${use_mock_hardware}">
+                    <plugin>mock_components/GenericSystem</plugin>
+                </xacro:if>
+                <xacro:unless value="${use_mock_hardware}">
+                    <plugin>piper_hardware/PiperSystem</plugin>
+                    <param name="feedback_topic">/joint_states</param>
+                    <param name="command_topic">/piper/joint_commands</param>
+                    <param name="ready_topic">/piper/hardware_ready</param>
+                    <param name="feedback_timeout">0.25</param>
+                    <param name="startup_timeout">5.0</param>
+                </xacro:unless>
             </hardware>
             <joint name="joint1">

File: src/piper_moveit/piper_no_gripper_moveit/config/piper.urdf.xacro (robot description, xacro)
@@ -1,4 +1,5 @@
 <?xml version="1.0"?>
 <robot xmlns:xacro="http://www.ros.org/wiki/xacro" name="piper">
+    <xacro:arg name="use_mock_hardware" default="false"/>
     <xacro:arg name="initial_positions_file" default="initial_positions.yaml" />
     <!-- Import piper urdf file -->
@@ -6,4 +7,4 @@
     <!-- Import control_xacro -->
     <xacro:include filename="piper.ros2_control.xacro" />
-    <xacro:piper_ros2_control name="FakeSystem" initial_positions_file="$(arg initial_positions_file)"/>
+    <xacro:piper_ros2_control name="PiperSystem" initial_positions_file="$(arg initial_positions_file)" use_mock_hardware="$(arg use_mock_hardware)"/>
 </robot>

File: src/piper_moveit/piper_no_gripper_moveit/config/piper_welding_gun.urdf.xacro (robot description, xacro)
@@ -1,10 +1,10 @@
 <?xml version="1.0"?>
 <robot xmlns:xacro="http://www.ros.org/wiki/xacro" name="piper">
+    <xacro:arg name="use_mock_hardware" default="false"/>
   <xacro:arg name="simulation" default="false"/>
   <xacro:arg name="initial_positions_file" default="$(find piper_no_gripper_moveit)/config/initial_positions.yaml"/>
   <xacro:include filename="$(find piper_description)/urdf/piper_welding_gun.urdf.xacro"/>
   <xacro:include filename="piper.ros2_control.xacro"/>
-  <!-- Same command bridge as the existing PiPER Real profile. The CAN driver
-       consumes local broadcaster setpoints and publishes measured /joint_states. -->
-  <xacro:piper_ros2_control name="PiperCommandBridge" initial_positions_file="$(arg initial_positions_file)"/>
+  <!-- Real CAN measurements feed the controller; commands use a separate topic. -->
+  <xacro:piper_ros2_control name="PiperCommandBridge" initial_positions_file="$(arg initial_positions_file)" use_mock_hardware="$(arg use_mock_hardware)"/>
 </robot>

File: src/piper_moveit/piper_with_gripper_moveit/config/piper.ros2_control.xacro (robot description, xacro)
@@ -1,10 +1,19 @@
 <?xml version="1.0"?>
 <robot xmlns:xacro="http://www.ros.org/wiki/xacro">
-    <xacro:macro name="piper_ros2_control" params="name initial_positions_file">
+    <xacro:macro name="piper_ros2_control" params="name initial_positions_file use_mock_hardware:=false">
         <xacro:property name="initial_positions" value="${load_yaml(initial_positions_file)['initial_positions']}"/>
         <ros2_control name="${name}" type="system">
             <hardware>
-                <!-- By default, set up controllers for simulation. This won't work on real hardware -->
-                <plugin>mock_components/GenericSystem</plugin>
+                <xacro:if value="${use_mock_hardware}">
+                    <plugin>mock_components/GenericSystem</plugin>
+                </xacro:if>
+                <xacro:unless value="${use_mock_hardware}">
+                    <plugin>piper_hardware/PiperSystem</plugin>
+                    <param name="feedback_topic">/joint_states</param>
+                    <param name="command_topic">/piper/joint_commands</param>
+                    <param name="ready_topic">/piper/hardware_ready</param>
+                    <param name="feedback_timeout">0.25</param>
+                    <param name="startup_timeout">5.0</param>
+                </xacro:unless>
             </hardware>
             <joint name="joint1">
@@ -55,5 +64,4 @@
                   <param name="initial_value">${initial_positions['joint7']}</param>
                 </state_interface>
-                <state_interface name="velocity"/>
             </joint>
             <joint name="joint8">
@@ -62,5 +70,4 @@
                   <param name="initial_value">${initial_positions['joint8']}</param>
                 </state_interface>
-                <state_interface name="velocity"/>
             </joint>
         </ros2_control>

File: src/piper_moveit/piper_with_gripper_moveit/config/piper.urdf.xacro (robot description, xacro)
@@ -1,4 +1,5 @@
 <?xml version="1.0"?>
 <robot xmlns:xacro="http://www.ros.org/wiki/xacro" name="piper">
+    <xacro:arg name="use_mock_hardware" default="false"/>
     <xacro:arg name="initial_positions_file" default="initial_positions.yaml" />
     <xacro:arg name="wrist_camera" default="oak_pro_w"/>
@@ -7,4 +8,4 @@
     <!-- Import control_xacro -->
     <xacro:include filename="piper.ros2_control.xacro" />
-    <xacro:piper_ros2_control name="FakeSystem" initial_positions_file="$(arg initial_positions_file)"/>
+    <xacro:piper_ros2_control name="PiperSystem" initial_positions_file="$(arg initial_positions_file)" use_mock_hardware="$(arg use_mock_hardware)"/>
 </robot>

File: src/robot_description/piper_description/urdf/include/piper_femto_bolt_handeye_macros.xacro (robot description, xacro)
@@ -1,5 +1,7 @@
 <?xml version="1.0"?>
 <!--
-  Piper + Orbbec Femto Bolt (eye-in-hand on link6).
+  Piper + Orbbec Femto Bolt (eye-in-hand; real mount on link5 since 2026-10-05,
+  simulation on link6). The real origin below is relative to that parent link and
+  is stale until the new mount is calibrated (robot_effector_frame:=link5).
   Frame names match orbbec_camera's femto_bolt.launch.py defaults (camera_name:=camera):
     camera_base_link, camera_link, camera_color_optical_frame, etc.
@@ -25,6 +27,6 @@
            mount is re-expressed using this camera's recorded driver extrinsics
            (2026-09-24); internal TFs themselves always come from the driver. -->
-      <origin xyz="${'-0.116960119269 0.004378100746 -0.028825832440' if use_nominal_extrinsics else '-0.116993388682 0.003847750737 -0.028481607579'}"
-              rpy="${'0.062955579669 -0.945517293938 -0.083284514853' if use_nominal_extrinsics else '0.062031929577 -0.945558883998 -0.082131313722'}"/>
+      <origin xyz="${'-0.116960119269 0.004378100746 -0.028825832440' if use_nominal_extrinsics else '-0.044525749544 -0.064654994020 -0.003299954006'}"
+              rpy="${'0.062955579669 -0.945517293938 -0.083284514853' if use_nominal_extrinsics else '1.698973335600 -0.016012269413 -1.559219138477'}"/>
     </xacro:femto_bolt>
   </xacro:macro>

File: src/robot_description/piper_description/urdf/piper_welding_gun.urdf.xacro (robot description, xacro)
@@ -4,46 +4,71 @@
   <xacro:arg name="simulation_controllers" default=""/>
   <xacro:arg name="wrist_camera" default="gazebo_realsense"/>
+  <!-- Real Femto Bolt mount since 2026-10-05 is on link5 (does not rotate with joint 6).
+       Simulation keeps link6 because its nominal extrinsics are expressed there. -->
+  <xacro:arg name="femto_parent_link" default="link5"/>
   <xacro:include filename="$(find piper_description)/urdf/piper_no_gripper_description_gz.xacro"/>
-  <!-- Adapter assembly STL: mm, mounting face at Z=0, CAD includes flange Z rotation. -->
+  <!-- AgileX PiPER flange (STL in mm): mounting face on link6 at Z=0, top recess Ø40.5 x 6 mm. -->
+  <link name="piper_flange">
+    <visual>
+      <geometry><mesh filename="package://piper_description/meshes/welding_gun/AgileX_PiPER_Flange.stl" scale="0.001 0.001 0.001"/></geometry>
+      <material name="piper_flange_metal"><color rgba="0.55 0.57 0.60 1"/></material>
+    </visual>
+    <!-- Real robot: end effector excluded from collision checking (operator request 2026-10-05). -->
+    <xacro:if value="$(arg simulation)">
+      <collision>
+        <geometry><mesh filename="package://piper_description/meshes/welding_gun/AgileX_PiPER_Flange.stl" scale="0.001 0.001 0.001"/></geometry>
+      </collision>
+    </xacro:if>
+    <inertial>
+      <origin xyz="0 0 0.0044"/>
+      <mass value="0.05"/>
+      <inertia ixx="0.00001" ixy="0" ixz="0" iyy="0.00001" iyz="0" izz="0.00002"/>
+    </inertial>
+  </link>
+  <joint name="piper_flange_mount" type="fixed">
+    <parent link="link6"/><child link="piper_flange"/>
+    <origin xyz="0 0 0" rpy="0 0 0"/>
+  </joint>
+  <!-- Welding gun frame stays identical to link6 so arm_tcp and calibrations keep their
+       values. The gun STL (mm) is modelled lying along -Y: its Ø39 spigot (y 47.8..54,
+       axis x=-5.85, z=28.5) sits in the flange recess, face y=47.8 on the flange top
+       (z=10.5 mm); the wire bend points to link6 +X, which matches the 2026-10-05 TCP
+       calibration within ~3.5 mm. -->
   <link name="piper_welding_gun">
     <visual>
-      <geometry><mesh filename="package://piper_description/meshes/welding_gun/PiPER_Prirubnica_Adapter_Welding_Gun.stl" scale="0.001 0.001 0.001"/></geometry>
+      <origin xyz="0.00585 -0.0285 0.0583" rpy="-1.5707963268 0 0"/>
+      <geometry><mesh filename="package://piper_description/meshes/welding_gun/03_welding_gun.stl" scale="0.001 0.001 0.001"/></geometry>
       <material name="piper_gun_metal"><color rgba="0.35 0.38 0.42 1"/></material>
     </visual>
-    <collision>
-      <geometry><mesh filename="package://piper_description/meshes/welding_gun/PiPER_Prirubnica_Adapter_Welding_Gun.stl" scale="0.001 0.001 0.001"/></geometry>
-    </collision>
+    <xacro:if value="$(arg simulation)">
+      <collision>
+        <origin xyz="0.00585 -0.0285 0.0583" rpy="-1.5707963268 0 0"/>
+        <geometry><mesh filename="package://piper_description/meshes/welding_gun/03_welding_gun.stl" scale="0.001 0.001 0.001"/></geometry>
+      </collision>
+    </xacro:if>
     <!-- Approximate prototype dynamics; no measured mass supplied with STL. -->
     <inertial>
-      <origin xyz="0.005 0 0.0775"/>
-      <mass value="0.45"/>
-      <inertia ixx="0.0016" ixy="0" ixz="0" iyy="0.0018" iyz="0" izz="0.0004"/>
+      <origin xyz="0.004 0 0.04"/>
+      <mass value="0.35"/>
+      <inertia ixx="0.0008" ixy="0" ixz="0" iyy="0.0008" iyz="0" izz="0.0003"/>
     </inertial>
   </link>
   <joint name="piper_welding_gun_mount" type="fixed">
-    <parent link="link6"/><child link="piper_welding_gun"/>
-    <!-- The assembly already includes the previous +90 degree flange Z rotation. -->
+    <parent link="piper_flange"/><child link="piper_welding_gun"/>
     <origin xyz="0 0 0" rpy="0 0 0"/>
   </joint>
-  <!-- TCP pivot/axis calibration 2026-09-23T14:02:51Z, parent link6.
-       Calibrated +Z is expressed as arm_tcp +X for the welding planner.
-       Position RMS 3.54 mm; independent physical validation is still required.
-       The gun mount is identity, so the flange-relative origin applies here. -->
+  <!-- Nominal CAD wire-tip TCP, applied 2026-09-30. TCP +X follows the wire. -->
   <link name="arm_tcp"/>
   <joint name="arm_tcp_joint" type="fixed">
     <parent link="piper_welding_gun"/><child link="arm_tcp"/>
-    <!-- Simulation: tip of the CAD wire/contact tip (end of the 3 mm stub), on the
-         35 deg bent nozzle axis (sin 35, 0, cos 35); TCP +X follows the wire. The
-         real robot keeps the calibrated pivot, which is not on the CAD axis. -->
-    <xacro:if value="$(arg simulation)">
-      <origin xyz="0.05360585785 0 0.2085160675" rpy="0 -0.9599310886 0"/>
-    </xacro:if>
-    <xacro:unless value="$(arg simulation)">
-      <origin xyz="0.059716507277 -0.002810430194 0.190158035855" rpy="-0.027929237913 -0.909524738174 0.022044250167"/>
-    </xacro:unless>
+    <!-- Wire tip of 03_welding_gun.stl on the AgileX flange (model geometry, 2026-10-05):
+         end-face centre of the Ø3 mm wire, axis 45.3 deg from link6 Z toward +X.
+         TCP +X follows the wire. Same for real robot and simulation. -->
+    <origin xyz="0.039746665881 -0.000003287520 0.111796185844" rpy="0 -0.7801056516 0"/>
   </joint>
   <xacro:if value="${'$(arg wrist_camera)' == 'femto_bolt'}">
     <xacro:include filename="$(find piper_description)/urdf/include/piper_femto_bolt_handeye_macros.xacro"/>
-    <xacro:piper_mount_femto_bolt_handeye parent_link="link6" use_nominal_extrinsics="$(arg simulation)"/>
+    <xacro:piper_mount_femto_bolt_handeye parent_link="${'link6' if '$(arg simulation)' == 'true' else '$(arg femto_parent_link)'}"
+                                         use_nominal_extrinsics="$(arg simulation)"/>
   </xacro:if>
   <xacro:unless value="${'$(arg wrist_camera)' == 'femto_bolt'}">
